File: uaefi-adapter-NA6.kicad_pcb (KiCad board)
At the start: 2 copper layers, 154 x 159 mm, 64 parts, among them J11 Conn_01x01, J13 Conn_01x01, J14 Conn_01x01, J15 Conn_01x01, J16 Conn_01x01, J17 Conn_01x01, P10 Pad, P15 Pad, P16 Pad, P17 Pad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

Commit message: upd
Other:
- board text added: "Always looking for C/C++/PHP/Java developers https://rusefi.com/s/mission"
- board text added: "COMMUNITY SUPPORT ECU https://rusefi.com/s/community https://rusefi.com/s/uaefi-NA"
- board text added: "FOR OFF ROAD PURPOSES ONLY This is not for applications with emissions or safety regulations (AKA not for street use). This is for closed stages, track and equipment."
Changed lines of the file:
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@@
     (fp_arc (start 96.474874 -99.974874) (mid 98.949755 -98.949755) (end 99.974874 -96.474874)
       (stroke (width 0.1) (type default)) (layer "F.SilkS"))
-    (fp_arc (start 99.974874 -3.474874) (mid 98.949737 -1.000026) (end 96.474874 0.025126)
+    (fp_arc (start 99.974874 -3.474874) (mid 98.949743 -0.999991) (end 96.474874 0.025126)
       (stroke (width 0.1) (type default)) (layer "F.SilkS"))
     (pad "A1" thru_hole roundrect (at 9.275 -25.8 90) (size 2.7 3.7) (drill 1.8) (layers "*.Cu" "*.Mask") (roundrect_rratio 0.092593)
@@
     (effects (font (size 1.016 1.016) (thickness 0.22352)) (justify mirror))
   )
+  (gr_text "Always looking for C/C++/PHP/Java developers\nhttps://rusefi.com/s/mission" (at 110 177.5) (layer "B.SilkS")
+    (effects (font (size 1.25 1.25) (thickness 0.25) bold) (justify left bottom mirror))
+  )
   (gr_text "4A" (at 72.935001 44.454999) (layer "B.SilkS")
     (effects (font (size 1.016 1.016) (thickness 0.22352)) (justify mirror))
@@
     (effects (font (size 1.016 0.8) (thickness 0.2)) (justify mirror))
   )
+  (gr_text "FOR OFF ROAD PURPOSES ONLY\nThis is not for applications with\nemissions or safety regulations\n(AKA not for street use). This is\nfor closed stages, track\nand equipment." (at 25 147.5 270) (layer "B.SilkS")
+    (effects (font (size 1.25 1.25) (thickness 0.25) bold) (justify left bottom mirror))
+  )
   (gr_text "3I" (at 133.200001 44.379999) (layer "B.SilkS")
     (effects (font (size 1.016 1.016) (thickness 0.22352)) (justify mirror))
@@
     (effects (font (size 0.8 0.7) (thickness 0.15)) (justify mirror))
   )
+  (gr_text "COMMUNITY SUPPORT ECU\nhttps://rusefi.com/s/community\nhttps://rusefi.com/s/uaefi-NA" (at 25 95 270) (layer "B.SilkS")
+    (effects (font (size 1.25 1.25) (thickness 0.25) bold) (justify left bottom mirror))
+  )
   (gr_text "1M" (at 55.015001 44.329999) (layer "B.SilkS")
     (effects (font (size 1.016 1.016) (thickness 0.22352)) (justify mirror))
@@
     (effects (font (size 0.508 0.508) (thickness 0.127)))
   )
+  (gr_text "FOR OFF ROAD PURPOSES ONLY\nThis is not for applications with\nemissions or safety regulations\n(AKA not for street use). This is\nfor closed stages, track\nand equipment." (at 25 117.5 270) (layer "F.SilkS")
+    (effects (font (size 1.25 1.25) (thickness 0.25) bold) (justify left bottom))
+  )
   (gr_text "3Q" (at 143.880001 42.399999 90) (layer "F.SilkS")
     (effects (font (size 0.508 0.508) (thickness 0.127)))
@@
     (effects (font (size 0.508 0.508) (thickness 0.127)))
   )
+  (gr_text "Always looking for C/C++/PHP/Java developers\nhttps://rusefi.com/s/mission" (at 80 177.5) (layer "F.SilkS")
+    (effects (font (size 1.25 1.25) (thickness 0.25) bold) (justify left bottom))
+  )
   (gr_text "2L" (at 107.431001 37.827999 90) (layer "F.SilkS")
     (effects (font (size 0.508 0.508) (thickness 0.127)))
@@
     (effects (font (size 0.508 0.508) (thickness 0.127)))
   )
+  (gr_text "COMMUNITY SUPPORT ECU\nhttps://rusefi.com/s/community\nhttps://rusefi.com/s/uaefi-NA" (at 25 65 -90) (layer "F.SilkS")
+    (effects (font (size 1.25 1.25) (thickness 0.25) bold) (justify left bottom))
+  )
   (gr_text "2I" (at 104.383001 42.399999 90) (layer "F.SilkS")

Commit message: upd
Parts:
- removed the P7 at (135.4, 82.6)
- removed the P7 at (132.9, 82.6)
- removed the P7 at (126.9, 82.6)
- removed the P7 at (126.9, 80.1)
- removed the P7 at (124.4, 80.1)
- removed the P7 at (132.9, 80.1)
- removed the P7 at (124.4, 82.6)
- removed the P7 at (135.4, 80.1)
