File: uaefi-adapter-NA6.kicad_pcb (KiCad board)
At the start: 2 copper layers, 154 x 159 mm, 56 parts, among them J11 Conn_01x01, J13 Conn_01x01, J14 Conn_01x01, J15 Conn_01x01, J16 Conn_01x01, J17 Conn_01x01, P10 Pad, P15 Pad, P16 Pad, P17 Pad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

Commit message: upd
Parts:
- added J1: 43045-0612, Connector_Molex:Molex_Micro-Fit_3.0_43045-0612_2x03_P3.00mm_Vertical, F.Cu at (210.3, 71.5)
- added Q1: ZXMS6005SGTA, Package_TO_SOT_SMD:SOT-223, F.Cu at (210.8, 82.9)
- P2: value 178780-1 -> Pad
- R18: value Jumper-Pad-Pad -> 750
- R21: value 1k -> Jumper-Pad-Pad
- R25: value Jumper-Pad-Pad -> 220
Connections:
- F2 pad 1: (no net) -> /1B
- F2 pad 2: (no net) -> /12V_FROM_MAIN_RELAY
- P10 pad 1: (no net) -> Net-(P10-Pin_1)
- P19 pad 1: (no net) -> /1P
- P2 pad 1: (no net) -> /1C
- P21 pad 1: (no net) -> Net-(P1A-1T)
- P3 pad 1: (no net) -> Net-(M1-DC1_DIR)
- P7 pad 1: (no net) -> Net-(M1-DC2_DIR)
- P8 pad 1: (no net) -> /1O
- P9 pad 1: (no net) -> Net-(M1-DC2_PWM)
- R12 pad 1: (no net) -> /IN_CLUTCH
- R12 pad 2: (no net) -> /1V
- R17 pad 1: (no net) -> /OUT_RADIATOR_FAN_RELAY
- R17 pad 2: (no net) -> /1L
- R18 pad 1: (no net) -> Net-(D1-K)
- R18 pad 2: (no net) -> /OUT_TACH
- R19 pad 1: (no net) -> /OUT_AC_RELAY
- R19 pad 2: (no net) -> /1J
- R21 pad 1: (no net) -> /OUT_IGN1
- R21 pad 2: (no net) -> /1G
- R22 pad 1: (no net) -> /CANL
- R22 pad 2: (no net) -> /1F
- R24 pad 1: (no net) -> /CANH
- R24 pad 2: (no net) -> /1D
- R25 pad 1: (no net) -> Net-(D1-A)
- R25 pad 2: (no net) -> /12V_FROM_MAIN_RELAY
- R28 pad 1: (no net) -> /OUT_PUMP_RELAY
- R28 pad 2: (no net) -> /3O
- R30 pad 1: (no net) -> /OUT_INJ4
- R30 pad 2: (no net) -> /3Z
- R31 pad 1: (no net) -> /OUT_INJ3
- R31 pad 2: (no net) -> /3Y
- R33 pad 1: (no net) -> /OUT_INJ4
- R33 pad 2: (no net) -> /OUT_INJ2
- R34 pad 1: (no net) -> /OUT_INJ3
- R34 pad 2: (no net) -> /OUT_INJ1
- R8 pad 1: (no net) -> /IN_TPS1
- R8 pad 2: (no net) -> Net-(P1D-4J)
Routing:
- net (no net): track 1371.7 -> 873.9 mm, vias 9 -> 7
- net /1B: track 0.00 -> 77.4 mm
- net /OUT_INJ3: track 0.00 -> 76.4 mm, vias 0 -> 1
- net /12V_FROM_MAIN_RELAY: track 0.00 -> 31.6 mm
- net /1L: track 0.00 -> 25.8 mm
- net Net-(P1D-4J): track 0.00 -> 24.8 mm
- net Net-(P10-Pin_1): track 0.00 -> 22.8 mm
- net /1V: track 0.00 -> 21.2 mm
- net Net-(P1A-1T): track 0.00 -> 19.4 mm
- net /OUT_TACH: track 0.00 -> 16.3 mm
- net Net-(M1-DC1_DIR): track 0.00 -> 15.6 mm
- net /1O: track 0.00 -> 15.1 mm
- net /3O: track 0.00 -> 14.9 mm
- net Net-(M1-DC2_PWM): track 0.00 -> 13.8 mm
- net /3Y: track 0.00 -> 12.4 mm
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