File: uaefi-adapter-NA6.kicad_sch (KiCad schematic)
At the start: 1 part

Commit message: upd
Parts:
- added P1: 178780-1, hellen-one-common:178780-1, symbol 178780-1:178780-1

Commit message: upd
Parts:
- added F1, F2, F3: Fuse-Pad-Pad, hellen-one-common:PAD-1206-PAD, symbol hellen-one-common:Fuse-Pad-Pad
- added P10, P11, P12, P2, P3, P4, P5, P6, P7, P8, P9: Pad, hellen-one-common:PAD-TH, symbol hellen-one-common:Pad
- added R1, R10, R11, R12, R13, R14, R15, R16, R17, R18, R19, R2, R20, R21, R22, R23, R24, R25, R26, R27, R28, R29, R3, R30, R31, R33, R34, R4, R5, R6, R7, R8, R9: Jumper-Pad-Pad, hellen-one-common:PAD-0805-PAD, symbol hellen-one-common:Jumper-Pad-Pad
- added R32: 1k, hellen-one-common:R0603, symbol hellen-one-common:Res
Connections:
- net at P1.65 (4A): now also P1.71 (4B)
- net at P1.66 (4C): now also P1.72 (4D)
- net GND: now reaches P1.67 (4E)
- net GND: now also P1.23 (2A), P1.28 (2K), P1.30 (2O), P1.39 (3A), P1.40 (3C), P1.52 (3B), P1.53 (3D), P1.73 (4F), R7.1
- net at P1.68 (4G): now also R11.2
- net at P1.69 (4I): now also R9.2
- net +5VAS: now reaches P1.70 (4K)
- net +5VAS: now also P1.31 (2B), P1.44 (3K), P1.76 (4L), R15.1
- net at P1.74 (4H): now also R10.2
- net at P1.75 (4J): now also R8.2
- net 2D: now reaches P1.32 (2D)
- net 2D: now also F1.1
- net 3I: now reaches P1.43 (3I)
- net 3I: now also R6.2
- net 3M: now reaches P1.45 (3M)
- net 3M: now also R4.2
- net 3O: now reaches P1.46 (3O)
- net 3O: now also R28.2, R29.2
- net 3S: now reaches P1.48 (3S)
- net 3S: now also R2.2
- net at P1.49 (3U): now also R34.2
- net 3Y: now reaches P1.51 (3Y)
- net 3Y: now also R31.2
- net 3F: now reaches P1.54 (3F)
- net 3F: now also R7.2
- net 3H: now reaches P1.55 (3H)
- net 3H: now also P3.1 (Pin_1)
- net 3J: now reaches P1.56 (3J)
- net 3J: now also P2.1 (Pin_1)
- net 3L: now reaches P1.57 (3L)
- net 3L: now also R5.2
- net 3N: now reaches P1.58 (3N)
- net 3N: now also R3.2
- net 3R: now reaches P1.60 (3R)
- net 3R: now also P5.1 (Pin_1)
- net 3T: now reaches P1.61 (3T)
- net 3T: now also R1.2
- net at P1.62 (3V): now also R33.2
- net 3X: now reaches P1.63 (3X)
- net 3X: now also P4.1 (Pin_1)
- net 3Z: now reaches P1.64 (3Z)
- net 3Z: now also R30.2
- net 1A: now reaches P1.1 (1A)
- net 1A: now also R25.2
- net at P1.10 (1S): now also P9.1 (Pin_1)
- net 1U: now reaches P1.11 (1U)
- net 1U: now also P7.1 (Pin_1)
- net 1B: now reaches P1.12 (1B)
- net 1B: now also F1.2, F2.1, F3.1
- net 1D: now reaches P1.13 (1D)
- net 1D: now also R24.2
- net 1F: now reaches P1.14 (1F)
- net 1F: now also R22.2
- net 1H: now reaches P1.15 (1H)
- net 1H: now also R20.2
- net 1J: now reaches P1.16 (1J)
- net 1J: now also R19.2
- net 1L: now reaches P1.17 (1L)
- net 1L: now also R17.2
- net 1N: now reaches P1.18 (1N)
- net 1N: now also R15.2
- net 1P: now reaches P1.19 (1P)
- net 1P: now also P10.1 (Pin_1)
- net 1C: now reaches P1.2 (1C)
- net 1C: now also P6.1 (Pin_1)
- net at P1.20 (1R): now also R13.2
- net at P1.21 (1T): now also P8.1 (Pin_1)
- net 1V: now reaches P1.22 (1V)
- net 1V: now also R12.2
- net 1E: now reaches P1.3 (1E)
- net 1E: now also R23.2
- net 1G: now reaches P1.4 (1G)
- net 1G: now also R21.2
- net at P1.5 (1I): now also P12.1 (Pin_1)
- net at P1.6 (1K): now also R18.2
- net 1M: now reaches P1.7 (1M)
- net 1M: now also R16.2
- net 1O: now reaches P1.8 (1O)
- net 1O: now also P11.1 (Pin_1)
- net 1Q: now reaches P1.9 (1Q)
- net 1Q: now also R14.2
- new net: R13.1, R17.1
- new net: R30.1, R33.1
- new net: R1.1, R28.1
- new net: R26.2, R27.1, R6.1
- new net: R27.2, R32.2
- new net: R4.1, R5.1
- new net: R31.1, R34.1
- new net +12V_ETB: F3.2
- new net +12V_PERM: R25.1
- new net +12V_PROT: R32.1
- new net +12V_RAW: F2.2
- no-connect marks 0 -> 1
Other:
- note added: "For 1990-1993"
- note added: "For 1990-1993 A/T and 1994+"
- note added: "For 1990-1993 M/T"
- note added: "For 1994+"
- note added: "Install R25 for 1990-1993 manual models with KIA TPS Also remove R22 for KIA TPS WARNING: Installing R25 with stock 1990-1993 TP switch will lead to short of 5V-GND!"
- note added: "Not OEM"
- note added: "Remove for KIA resistive TP Sensor"

Commit message: upd
Parts:
- added P13, P14, P15, P16, P17, P18, P19, P20: Pad, hellen-one-common:PAD-TH, symbol hellen-one-common:Pad
Connections:
- net OUT_ECF_RELAY: now reaches R13.1, R17.1
- net IN_VSS: now reaches R16.1
- net IN_MAF: now reaches R29.1
- net OUT_IGN1: now reaches R21.1
- net CAN-: now reaches R22.1
- net at BRD1.D13 (IN_TPS1): now also P17.1 (Pin_1)
- net at BRD1.D14 (IN_KNOCK_RAW): now also P18.1 (Pin_1)
- net at BRD1.D15 (IN_IAT): now also P19.1 (Pin_1)
- net at BRD1.D16 (IN_CLT): now also P20.1 (Pin_1)
- net at BRD1.D5 (IN_FLEX): now also P13.1 (Pin_1)
- net at BRD1.D6 (IN_PPS1): now also P14.1 (Pin_1)
- net at BRD1.D7 (CAN+): now also P15.1 (Pin_1)
- net at BRD1.D8 (CAN-): now also P16.1 (Pin_1)
- net IN_CRANK: now reaches P1.41 (3E)
- net IN_CAM: now reaches P1.42 (3G)
- net IN_CLT: now reaches P1.47 (3Q)
- net OUT_INJ1: now reaches P1.49 (3U), R34.2
- net OUT_IDLE: now reaches P1.50 (3W)
- net IN_IAT: now reaches P1.59 (3P)
- net OUT_INJ2: now reaches P1.62 (3V), R33.2
- net IN_TPS: now reaches R8.1
- net IN_TPS: now also R4.1, R5.1
- net OUT_INJ4: now reaches R30.1, R33.1
- net IN_PPS: now reaches R9.1
- net OUT_AC_RELAY: now reaches R19.1
- net OUT_IGN2: now reaches R20.1
- net OUT_PUMP_RELAY: now reaches R1.1, R28.1
- net OUT_CHECK_ENGINE: now reaches R23.1
- net IN_AC_SW: now reaches R14.1
- net IN_O2S: now reaches R3.1
- net IN_TEMP_OR_PPS2: now reaches R11.1
- net OUT_CONDENSER_FAN: now reaches R2.1
- net OUT_ETB+: now reaches P1.65 (4A), P1.71 (4B)
- net OUT_ETB-: now reaches P1.66 (4C), P1.72 (4D)
- net IN_TPS2: now reaches R10.1
- net OUT_TACH: now reaches R26.1
- net OUT_INJ3: now reaches R31.1, R34.1
- net CAN+: now reaches R24.1
- net IN_CLUTCH: now reaches R12.1
- net WBO_H-: now reaches P1.24 (2C)
- net WBO_R_Trim: now reaches P1.25 (2E)
- net WBO_Vs/Ip: now reaches P1.26 (2G)
- net OUT_VVT: now reaches P1.27 (2I)
- net IN_PRESSURE: now reaches P1.29 (2M)
- net WBO_Ip: now reaches P1.33 (2F)
- net WBO_Vs: now reaches P1.34 (2H)
- net OUT_BOOST_CONTROL: now reaches P1.35 (2J)
- net IN_DIGITAL: now reaches P1.36 (2L)
- net IN_TEMP: now reaches P1.37 (2N)
- net IN_KNOCK_RAW: now reaches P1.38 (2P)

Commit message: upd
Connections:
- net CAN+: now also BRD1.D7 (CAN+), P15.1 (Pin_1)
- net CAN-: now also BRD1.D8 (CAN-), P16.1 (Pin_1)
- net GND: now also BRD1.C12 (GNDA), BRD1.C13 (GNDA)
- net IN_CLT: now also BRD1.D16 (IN_CLT), P20.1 (Pin_1)
- net IN_IAT: now also BRD1.D15 (IN_IAT), P19.1 (Pin_1)
- net IN_KNOCK_RAW: now also BRD1.D14 (IN_KNOCK_RAW), P18.1 (Pin_1)
- net IN_TEMP_OR_PPS2: now also BRD1.C4 (IN_PPS2)
- net IN_TPS: now also BRD1.D13 (IN_TPS1), P17.1 (Pin_1)
- net IN_TPS2: now also BRD1.C14 (IN_TPS2)
- net OUT_CONDENSER_FAN: now also BRD1.B8 (OUT_LS_WEAK2)
- net OUT_IDLE: now also BRD1.B18 (OUT_LS2)
- net OUT_IGN1: now also BRD1.B15 (OUT_IGN1)
- net OUT_IGN2: now also BRD1.B14 (OUT_IGN2)
- net OUT_INJ1: now also BRD1.B6 (OUT_INJ1)
- net OUT_INJ2: now also BRD1.B5 (OUT_INJ2)
- net OUT_INJ3: now also BRD1.B4 (OUT_INJ3)
- net OUT_INJ4: now also BRD1.B3 (OUT_INJ4)
- net OUT_PUMP_RELAY: now also BRD1.B16 (OUT_LS4)
Other:
- note added: "!!!!"
- note added: "Fan Relay"
- note added: "Fuel Pump Relay"
- note added: "Idle Air Valve"
- note added: "Main Relay"
- note added: "OK"
- moved on the sheet: P13, P14, P15, P16, P17, P18, P19, P20

Commit message: upd
Connections:
- net +12V_RAW: now also BRD1.E1 (+12V_RAW)
- net 1B: now also BRD1.B1 (OUT_INJ6)
- net GND: now also BRD1.A3 (GND), BRD1.A4 (GND), BRD1.C11 (GNDA), BRD1.C8 (GND), BRD1.D11 (GNDA), BRD1.D12 (GNDA)
- net CAM1: now reaches BRD1.C5 (IN_HALL1)
- net CAM2: now reaches BRD1.C6 (IN_HALL2)
Other:
- note added: "CAM1"
- note added: "CAM2"
- note added: "VVT1"
- moved on the sheet: BRD1

Commit message: upd
Connections:
- net GND: now also BRD1.J4 (GND), BRD1.J5 (GND)
Changed lines of the file:
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@@
   (junction (at 138.43 87.63) (diameter 0) (color 0 0 0 0)
   )
+  (junction (at 334.01 220.98) (diameter 0) (color 0 0 0 0)
+  )
   (junction (at 102.87 102.87) (diameter 1.016) (color 0 0 0 0)
   )
@@
     (stroke (width 0) (type solid))
   )
+  (wire (pts (xy 334.01 220.98) (xy 347.98 220.98))
+    (stroke (width 0) (type default))
+  )
   (wire (pts (xy 347.98 109.22) (xy 307.34 109.22))
     (stroke (width 0) (type default))
@@
     (stroke (width 0) (type default))
   )
+  (wire (pts (xy 334.01 218.44) (xy 334.01 220.98))
+    (stroke (width 0) (type default))
+  )
   (wire (pts (xy 307.34 160.02) (xy 347.98 160.02))
     (stroke (width 0) (type default))
@@
     (stroke (width 0) (type solid))
   )
+  (wire (pts (xy 307.34 220.98) (xy 334.01 220.98))
+    (stroke (width 0) (type default))
+  )
   (wire (pts (xy 67.31 45.72) (xy 152.4 45.72))
     (stroke (width 0) (type default))
@@
     (stroke (width 0) (type default))
   )
+  (wire (pts (xy 347.98 218.44) (xy 334.01 218.44))
+    (stroke (width 0) (type default))
+  )
   (wire (pts (xy 85.09 236.22) (xy 85.09 233.68))
     (stroke (width 0) (type default))
@@
     (effects (font (size 2 2) (color 23 135 61 1)) (justify left bottom))
   )
+  (text "!!!!" (at 154.94 118.11 0)
+    (effects (font (size 2 2) (color 255 0 28 1)) (justify left bottom))
+  )
   (text "!!!!" (at 153.67 51.435 0)
     (effects (font (size 2 2) (color 255 0 28 1)) (justify left bottom))
@@
     (effects (font (size 2 2) (color 255 0 28 1)) (justify left bottom))
   )
-  (text "OK" (at 154.94 118.11 0)
-    (effects (font (size 2 2) (color 23 135 61 1)) (justify left bottom))
-  )
   (text "CAM1" (at 372.11 106.68 0)
     (effects (font (size 1.27 1.27)) (justify left bottom))
@@
         )
       )
+    )
+  )
+  (symbol (lib_id "power:GND") (at 307.34 220.98 270) (mirror x) (unit 1)
+    (in_bom yes) (on_board yes) (dnp no)
+    (property "Reference" "#PWR022" (at 300.99 220.98 0)
+      (effects (font (size 1.27 1.27)) hide)
+    )
+    (property "Value" "GND" (at 302.895 220.98 90)
+      (effects (font (size 1.27 1.27)))
+    )
+    (property "Footprint" "" (at 307.34 220.98 0)
+      (effects (font (size 1.27 1.27)) hide)
+    )
+    (property "Datasheet" "" (at 307.34 220.98 0)
+      (effects (font (size 1.27 1.27)) hide)
+    )
+    (pin "1")
+    (instances
+      (project "uaefi-adapter-NA6"
+        (path "/62be380c-4f45-483a-9614-39f0039d587a"
+          (reference "#PWR022") (unit 1)
+        )
+      )
+      (project "hellen64_NA6_94"
+        (path "/63d2dd9f-d5ff-4811-a88d-0ba932475460"
+          (reference "#PWR0101") (unit 1)
+        )
+      )

Commit message: upd
Parts:
- removed BRD1: uaefi, uaefi_brd:UAEFI_BRD, symbol uaefi_brd:UAEFI_BRD
- added BRD2: uaefi, uaefi_brd:UAEFI_BRD, symbol uaefi_brd:UAEFI_BRD
Connections:
- net +12V_RAW: now also BRD2.E1 (+12V_RAW)
- net 1B: now also BRD2.B1 (OUT_INJ6)
- net CAM1: now also BRD2.C5 (IN_HALL1)
- net CAM2: now also BRD2.C6 (IN_HALL2)
- net CAN+: now also BRD2.D7 (CAN+)
- net CAN-: now also BRD2.D8 (CAN-)
- net GND: now also BRD2.A3 (GND), BRD2.A4 (GND), BRD2.C8 (GND), BRD2.J4 (GND), BRD2.J5 (GND); no longer P1.40 (3C), P1.52 (3B), P1.53 (3D), P1.67 (4E), P1.73 (4F), R7.1
- net IN_CLT: now also BRD2.D16 (IN_CLT)
- net IN_IAT: now also BRD2.D15 (IN_IAT)
- net IN_KNOCK_RAW: now also BRD2.D14 (IN_KNOCK_RAW)
- net IN_TEMP_OR_PPS2: now also BRD2.C4 (IN_PPS2)
- net IN_TPS: now also BRD2.D13 (IN_TPS1)
- net IN_TPS2: now also BRD2.C14 (IN_TPS2)
- net OUT_CONDENSER_FAN: now also BRD2.B8 (OUT_LS_WEAK2)
- net OUT_IDLE: now also BRD2.B18 (OUT_LS2)
- net OUT_IGN1: now also BRD2.B15 (OUT_IGN1)
- net OUT_IGN2: now also BRD2.B14 (OUT_IGN2)
- net OUT_INJ1: now also BRD2.B6 (OUT_INJ1)
- net OUT_INJ2: now also BRD2.B5 (OUT_INJ2)
- net OUT_INJ3: now also BRD2.B4 (OUT_INJ3)
- net OUT_INJ4: now also BRD2.B3 (OUT_INJ4)
- net OUT_PUMP_RELAY: now also BRD2.B16 (OUT_LS4)
- net at P13.1 (Pin_1): now also BRD2.D5 (IN_FLEX)
- net at P14.1 (Pin_1): now also BRD2.D6 (IN_PPS1)
- new net GNDA: BRD2.C11 (GNDA), BRD2.C12 (GNDA), BRD2.C13 (GNDA), BRD2.D11 (GNDA), BRD2.D12 (GNDA), P1.40 (3C), P1.52 (3B), P1.53 (3D), P1.67 (4E), P1.73 (4F), R7.1
Other:
- note removed: "CAM1"
- note removed: "CAM2"
- note removed: "Fan Relay"
- note removed: "Fuel Pump Relay"
- note removed: "Idle Air Valve"
- note removed: "Main Relay"
- note removed: "VVT1"

Commit message: upd
Connections:
- net CAM1 is gone; now on net IN_CAM: BRD2.C5 (IN_HALL1)
- net CAM2 is gone; now on net IN_CRANK: BRD2.C6 (IN_HALL2)
- net +12V_RAW: now also BRD2.A7 (F1), BRD2.A8 (F2)
- net IN_AC_SW: now also BRD2.D10 (IN_BUTTON2)
- net IN_CLUTCH: now also BRD2.D2 (IN_BUTTON1)
- net IN_DIGITAL: now also BRD2.D5 (IN_FLEX), P13.1 (Pin_1)
- net IN_PRESSURE: now also BRD2.C15 (IN_AUX3)
- net OUT_BOOST_CONTROL: now also BRD2.B2 (OUT_INJ5)
- net OUT_ECF_RELAY renamed OUT_RADIATOR_FAN_RELAY
Changed lines of the file:
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@@
     (stroke (width 0) (type solid))
+  )
+  (wire (pts (xy 307.34 40.64) (xy 307.34 43.18))
+    (stroke (width 0) (type default))
   )
   (wire (pts (xy 111.76 130.81) (xy 67.31 130.81))
@@
     (effects (font (size 2 2) (color 255 0 28 1)) (justify left bottom))
   )
+  (text "OK" (at 154.94 197.485 0)
+    (effects (font (size 2 2) (color 23 135 61 1)) (justify left bottom))
+  )
   (text "OK" (at 154.94 93.98 0)
     (effects (font (size 2 2) (color 23 135 61 1)) (justify left bottom))
@@
     (effects (font (size 2 2) (color 23 135 61 1)) (justify left bottom))
   )
-  (text "!!!!" (at 154.94 128.27 0)
-    (effects (font (size 2 2) (color 255 0 28 1)) (justify left bottom))
-  )
   (text "OK" (at 139.065 200.025 0)
     (effects (font (size 2 2) (color 23 135 61 1)) (justify left bottom))
@@
     (effects (font (size 2 2) (color 23 135 61 1)) (justify left bottom))
   )
+  (text "OK" (at 153.67 40.64 0)
+    (effects (font (size 2 2) (color 23 135 61 1)) (justify left bottom))
+  )
+  (text "OK" (at 154.94 128.27 0)
+    (effects (font (size 2 2) (color 23 135 61 1)) (justify left bottom))
+  )
   (text "!!!!" (at 153.67 30.48 0)
     (effects (font (size 2 2) (color 255 0 28 1)) (justify left bottom))
   )
+  (text "OK" (at 154.94 149.225 0)
+    (effects (font (size 2 2) (color 23 135 61 1)) (justify left bottom))
+  )
   (text "!!!!" (at 153.67 45.72 0)
     (effects (font (size 2 2) (color 255 0 28 1)) (justify left bottom))
@@
     (effects (font (size 2 2) (color 255 0 28 1)) (justify left bottom))
   )
-  (text "!!!!" (at 154.94 161.29 0)
-    (effects (font (size 2 2) (color 255 0 28 1)) (justify left bottom))
-  )
   (text "OK" (at 154.94 74.93 0)
     (effects (font (size 2 2) (color 23 135 61 1)) (justify left bottom))
@@
     (effects (font (size 2 2) (color 23 135 61 1)) (justify left bottom))
   )
+  (text "OK" (at 154.94 161.29 0)
+    (effects (font (size 2 2) (color 23 135 61 1)) (justify left bottom))
+  )
   (text "!!!!" (at 154.94 118.11 0)
     (effects (font (size 2 2) (color 255 0 28 1)) (justify left bottom))
@@
     (effects (font (size 2 2) (color 23 135 61 1)) (justify left bottom))
   )
-  (text "!!!!" (at 154.94 123.19 0)
-    (effects (font (size 2 2) (color 255 0 28 1)) (justify left bottom))
-  )
-  (text "!!!!" (at 154.94 148.59 0)
-    (effects (font (size 2 2) (color 255 0 28 1)) (justify left bottom))
-  )
   (text "OK" (at 154.94 184.15 0)
     (effects (font (size 2 2) (color 23 135 61 1)) (justify left bottom))
@@
     (effects (font (size 1.27 1.27)) (justify left bottom))
   )
+  (text "OK" (at 153.67 36.195 0)
+    (effects (font (size 2 2) (color 23 135 61 1)) (justify left bottom))
+  )
   (text "Not OEM" (at 106.68 194.31 0)
     (effects (font (size 1.27 1.27)) (justify left bottom))
@@
   )
   (text "!!!!" (at 154.94 191.77 0)
-    (effects (font (size 2 2) (color 255 0 28 1)) (justify left bottom))
-  )
-  (text "!!!!" (at 153.67 35.56 0)
     (effects (font (size 2 2) (color 255 0 28 1)) (justify left bottom))
   )
@@
     (effects (font (size 1.27 1.27)) (justify left bottom))
   )
-  (text "!!!!" (at 153.67 33.02 0)
-    (effects (font (size 2 2) (color 255 0 28 1)) (justify left bottom))
-  )
   (text "For 1994+\n" (at 115.57 102.87 0)
     (effects (font (size 1.27 1.27)) (justify left bottom))
@@
     (effects (font (size 2 2) (color 23 135 61 1)) (justify left bottom))
   )
-  (text "!!!!" (at 154.94 196.85 0)
-    (effects (font (size 2 2) (color 255 0 28 1)) (justify left bottom))
-  )
   (text "For 1994+" (at 87.63 92.71 0)
     (effects (font (size 1.27 1.27)) (justify left bottom))
@@
     (effects (font (size 2 2) (color 255 0 28 1)) (justify left bottom))
   )
+  (text "OK" (at 154.94 123.19 0)
+    (effects (font (size 2 2) (color 23 135 61 1)) (justify left bottom))
+  )
   (text "OK" (at 154.94 107.95 0)
     (effects (font (size 2 2) (color 23 135 61 1)) (justify left bottom))
@@
     (effects (font (size 2 2) (color 255 0 28 1)) (justify left bottom))
   )
+  (text "OK" (at 153.67 33.02 0)
+    (effects (font (size 2 2) (color 23 135 61 1)) (justify left bottom))
+  )
   (text "OK" (at 154.94 226.06 0)
     (effects (font (size 2 2) (color 23 135 61 1)) (justify left bottom))
@@
     (effects (font (size 2 2) (color 255 0 28 1)) (justify left bottom))
   )
-  (text "!!!!" (at 153.67 40.64 0)
-    (effects (font (size 2 2) (color 255 0 28 1)) (justify left bottom))
-  )
   (label "OUT_IGN2" (at 307.34 81.28 180) (fields_autoplaced)
     (effects (font (size 1.27 1.27)) (justify right bottom))
@@
     (effects (font (size 1.27 1.27)) (justify left bottom))
   )
+  (label "IN_AC_SW" (at 307.34 172.72 180) (fields_autoplaced)
+    (effects (font (size 1.27 1.27)) (justify right bottom))
+  )
   (label "IN_AC_SW" (at 152.4 161.29 180) (fields_autoplaced)
     (effects (font (size 1.27 1.27)) (justify right bottom))
@@
     (effects (font (size 1.27 1.27)) (justify right bottom))
   )
+  (label "IN_CAM" (at 307.34 106.68 180) (fields_autoplaced)
+    (effects (font (size 1.27 1.27)) (justify right bottom))
+  )
   (label "IN_TPS2" (at 152.4 223.52 180) (fields_autoplaced)
     (effects (font (size 1.27 1.27)) (justify right bottom))
@@
     (effects (font (size 1.27 1.27)) (justify left bottom))
   )
-  (label "CAM1" (at 307.34 106.68 180) (fields_autoplaced)
-    (effects (font (size 1.27 1.27)) (justify right bottom))
-  )
   (label "WBO_Vs" (at 152.4 45.72 180) (fields_autoplaced)
     (effects (font (size 1.27 1.27)) (justify right bottom))
@@
     (effects (font (size 1.27 1.27)) (justify left bottom))
   )
+  (label "IN_CRANK" (at 307.34 109.22 180) (fields_autoplaced)
+    (effects (font (size 1.27 1.27)) (justify right bottom))
+  )
   (label "OUT_PUMP_RELAY" (at 152.4 90.17 180) (fields_autoplaced)
     (effects (font (size 1.27 1.27)) (justify right bottom))
   )
+  (label "OUT_BOOST_CONTROL" (at 307.34 50.8 180) (fields_autoplaced)
+    (effects (font (size 1.27 1.27)) (justify right bottom))
+  )
   (label "IN_TEMP_OR_PPS2" (at 152.4 226.06 180) (fields_autoplaced)
     (effects (font (size 1.27 1.27)) (justify right bottom))
@@
     (effects (font (size 1.27 1.27)) (justify right bottom))
   )
-  (label "CAM2" (at 307.34 109.22 180) (fields_autoplaced)
-    (effects (font (size 1.27 1.27)) (justify right bottom))
-  )
   (label "3B" (at 88.9 135.89 0) (fields_autoplaced)
     (effects (font (size 1.27 1.27)) (justify left bottom))
@@
     (effects (font (size 1.27 1.27)) (justify right bottom))
   )
+  (label "IN_V_MAIN" (at 307.34 43.18 180) (fields_autoplaced)
+    (effects (font (size 1.27 1.27)) (justify right bottom))
+  )
   (label "OUT_CHECK_ENGINE" (at 152.4 191.77 180) (fields_autoplaced)
     (effects (font (size 1.27 1.27)) (justify right bottom))
@@
     (effects (font (size 1.27 1.27)) (justify left bottom))
   )
+  (label "IN_VIGN" (at 307.34 40.64 180) (fields_autoplaced)
+    (effects (font (size 1.27 1.27)) (justify right bottom))
+  )
   (label "3H" (at 72.39 120.65 0) (fields_autoplaced)
     (effects (font (size 1.27 1.27)) (justify left bottom))
@@
     (effects (font (size 1.27 1.27)) (justify left bottom))
   )
+  (label "IN_PRESSURE" (at 307.34 132.08 180) (fields_autoplaced)
+    (effects (font (size 1.27 1.27)) (justify right bottom))
+  )
   (label "OUT_INJ3" (at 152.4 77.47 180) (fields_autoplaced)
     (effects (font (size 1.27 1.27)) (justify right bottom))
@@
     (effects (font (size 1.27 1.27)) (justify left bottom))
   )
+  (label "IN_CLUTCH" (at 307.34 152.4 180) (fields_autoplaced)
+    (effects (font (size 1.27 1.27)) (justify right bottom))
+  )
   (label "IN_CRANK" (at 152.4 128.27 180) (fields_autoplaced)
     (effects (font (size 1.27 1.27)) (justify right bottom))
@@
     (effects (font (size 1.27 1.27)) (justify right bottom))
   )
-  (label "OUT_ECF_RELAY" (at 152.4 173.99 180) (fields_autoplaced)
+  (label "OUT_RADIATOR_FAN_RELAY" (at 152.4 173.99 180) (fields_autoplaced)
     (effects (font (size 1.27 1.27)) (justify right bottom))
   )
@@
     (effects (font (size 1.27 1.27)) (justify right bottom))
   )
+  (label "IN_DIGITAL" (at 316.865 160.02 180) (fields_autoplaced)
+    (effects (font (size 1.27 1.27)) (justify right bottom))
+  )
