File: uaefi-adapter-NA6.kicad_sch (KiCad schematic)
At the start: 58 parts, among them P1 178780-1, P10 Pad, P11 Pad, P12 Pad, P13 Pad, P14 Pad, P15 Pad, P16 Pad, P17 Pad, P18 Pad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

Commit message: upd
Connections:
- net 1B: no longer BRD2.B1 (OUT_INJ6)
Changed lines of the file:
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@@
     (stroke (width 0) (type solid))
-  )
-  (wire (pts (xy 347.98 48.26) (xy 307.34 48.26))
-    (stroke (width 0) (type default))
   )
   (wire (pts (xy 105.41 171.45) (xy 152.4 171.45))
@@
     (effects (font (size 1.27 1.27)) (justify right bottom))
   )
-  (label "1B" (at 307.34 48.26 180) (fields_autoplaced)
-    (effects (font (size 1.27 1.27)) (justify right bottom))
-  )

Commit message: upd
Parts:
- renumbered BRD2 to BRD?
Connections:
- net OUT_CONDENSER_FAN: now also BRD?.B1 (OUT_INJ6); no longer BRD?.B8 (OUT_LS_WEAK2)
- net OUT_RADIATOR_FAN_RELAY: now also BRD?.B8 (OUT_LS_WEAK2)
Changed lines of the file:
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@@
-    (stroke (width 0) (type default))
-  )
-  (wire (pts (xy 347.98 38.1) (xy 307.34 38.1))
     (stroke (width 0) (type default))
   )
@@
     (stroke (width 0) (type default))
   )
+  (wire (pts (xy 307.34 40.64) (xy 307.34 43.18))
+    (stroke (width 0) (type default))
+  )
   (wire (pts (xy 96.52 156.21) (xy 69.85 156.21))
     (stroke (width 0) (type solid))
@@
     (stroke (width 0) (type solid))
   )
-  (wire (pts (xy 347.98 35.56) (xy 307.34 35.56))
-    (stroke (width 0) (type default))
-  )
   (wire (pts (xy 347.98 203.2) (xy 307.34 203.2))
     (stroke (width 0) (type default))
@@
     (stroke (width 0) (type default))
   )
+  (wire (pts (xy 347.98 48.26) (xy 307.34 48.26))
+    (stroke (width 0) (type default))
+  )
   (wire (pts (xy 124.46 199.39) (xy 120.65 199.39))
     (stroke (width 0) (type solid))
@@
   (wire (pts (xy 67.31 184.15) (xy 95.25 184.15))
     (stroke (width 0) (type solid))
-  )
-  (wire (pts (xy 307.34 40.64) (xy 307.34 43.18))
-    (stroke (width 0) (type default))
   )
   (wire (pts (xy 111.76 130.81) (xy 67.31 130.81))
@@
     (effects (font (size 2 2) (color 23 135 61 1)) (justify left bottom))
   )
+  (text "OK" (at 154.94 174.625 0)
+    (effects (font (size 2 2) (color 23 135 61 1)) (justify left bottom))
+  )
   (text "OK" (at 139.065 200.025 0)
     (effects (font (size 2 2) (color 23 135 61 1)) (justify left bottom))
@@
     (effects (font (size 1.27 1.27)) (justify left bottom))
   )
-  (text "!!!!" (at 154.94 173.99 0)
-    (effects (font (size 2 2) (color 255 0 28 1)) (justify left bottom))
-  )
   (text "!!!!" (at 154.94 191.77 0)
     (effects (font (size 2 2) (color 255 0 28 1)) (justify left bottom))
@@
     (effects (font (size 1.27 1.27)) (justify left bottom))
   )
+  (label "OUT_RADIATOR_FAN_RELAY" (at 307.34 66.04 180) (fields_autoplaced)
+    (effects (font (size 1.27 1.27)) (justify right bottom))
+  )
   (label "IN_KNOCK_RAW" (at 152.4 25.4 180) (fields_autoplaced)
     (effects (font (size 1.27 1.27)) (justify right bottom))
@@
     (effects (font (size 1.27 1.27)) (justify right bottom))
   )
+  (label "OUT_CONDENSER_FAN" (at 307.34 48.26 180) (fields_autoplaced)
+    (effects (font (size 1.27 1.27)) (justify right bottom))
+  )
   (label "IN_DIGITAL" (at 316.865 160.02 180) (fields_autoplaced)
     (effects (font (size 1.27 1.27)) (justify right bottom))
   )
   (label "OUT_ETB+" (at 152.4 238.76 180) (fields_autoplaced)
-    (effects (font (size 1.27 1.27)) (justify right bottom))
-  )
-  (label "OUT_CONDENSER_FAN" (at 307.34 66.04 180) (fields_autoplaced)
     (effects (font (size 1.27 1.27)) (justify right bottom))
   )
@@
     )
   )
-  (symbol (lib_name "UAEFI_BRD_1") (lib_id "uaefi_brd:UAEFI_BRD") (at 347.98 25.4 0) (unit 1)
-    (in_bom yes) (on_board yes) (dnp no)
-    (property "Reference" "BRD2" (at 355.6 20.955 0)
+  (symbol (lib_id "uaefi_brd:UAEFI_BRD") (at 347.98 25.4 0) (unit 1)
+    (in_bom yes) (on_board yes) (dnp no)
+    (property "Reference" "BRD?" (at 355.6 20.955 0)
       (effects (font (size 1.27 1.27)) (justify left))
     )
@@
       (project "uaefi-adapter-NA6"
         (path "/62be380c-4f45-483a-9614-39f0039d587a"
-          (reference "BRD2") (unit 1)
-        )
-      )
+          (reference "BRD?") (unit 1)
+        )
+      )

Commit message: upd
Parts:
- removed P13, P14, P15, P16, P17, P18, P19, P20: Pad, hellen-one-common:PAD-TH, symbol hellen-one-common:Pad

Commit message: upd
Connections:
- net IN_O2S: now also BRD?.C3 (IN_AUX2)
- net IN_PPS: now also BRD?.D6 (IN_PPS1)
- net IN_TEMP: now also BRD?.D1 (IN_AUX1)
- net IN_VSS: now also BRD?.C7 (IN_HALL3)
- net OUT_TACH: now also BRD?.B10 (OUT_IGN6)
Changed lines of the file:
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@@
     (stroke (width 0) (type default))
   )
-  (text "!!!!" (at 154.94 171.45 0)
-    (effects (font (size 2 2) (color 255 0 28 1)) (justify left bottom))
-  )
   (text "OK" (at 154.94 197.485 0)
     (effects (font (size 2 2) (color 23 135 61 1)) (justify left bottom))
@@
     (effects (font (size 2 2) (color 23 135 61 1)) (justify left bottom))
   )
-  (text "!!!!" (at 153.67 30.48 0)
-    (effects (font (size 2 2) (color 255 0 28 1)) (justify left bottom))
-  )
   (text "OK" (at 154.94 149.225 0)
     (effects (font (size 2 2) (color 23 135 61 1)) (justify left bottom))
@@
     (effects (font (size 2 2) (color 23 135 61 1)) (justify left bottom))
   )
+  (text "OK" (at 154.94 118.11 0)
+    (effects (font (size 2 2) (color 23 135 61 1)) (justify left bottom))
+  )
   (text "OK" (at 102.87 231.14 0)
     (effects (font (size 2 2) (color 23 135 61 1)) (justify left bottom))
@@
     (effects (font (size 2 2) (color 23 135 61 1)) (justify left bottom))
   )
-  (text "!!!!" (at 154.94 118.11 0)
-    (effects (font (size 2 2) (color 255 0 28 1)) (justify left bottom))
-  )
   (text "!!!!" (at 153.67 51.435 0)
     (effects (font (size 2 2) (color 255 0 28 1)) (justify left bottom))
@@
     (effects (font (size 2 2) (color 255 0 28 1)) (justify left bottom))
   )
+  (text "OK" (at 154.94 171.45 0)
+    (effects (font (size 2 2) (color 23 135 61 1)) (justify left bottom))
+  )
   (text "OK" (at 154.94 82.55 0)
     (effects (font (size 2 2) (color 23 135 61 1)) (justify left bottom))
@@
   (text "!!!!" (at 154.94 102.87 0)
     (effects (font (size 2 2) (color 255 0 28 1)) (justify left bottom))
+  )
+  (text "OK" (at 154.94 105.41 0)
+    (effects (font (size 2 2) (color 23 135 61 1)) (justify left bottom))
   )
   (text "For 1990-1993\n" (at 104.14 158.75 0)
@@
     (effects (font (size 2 2) (color 23 135 61 1)) (justify left bottom))
   )
-  (text "!!!!" (at 154.94 220.98 0)
-    (effects (font (size 2 2) (color 255 0 28 1)) (justify left bottom))
+  (text "OK" (at 153.67 30.48 0)
+    (effects (font (size 2 2) (color 23 135 61 1)) (justify left bottom))
   )
   (text "OK" (at 154.94 123.19 0)
@@
     (effects (font (size 2 2) (color 23 135 61 1)) (justify left bottom))
   )
-  (text "!!!!" (at 154.94 105.41 0)
-    (effects (font (size 2 2) (color 255 0 28 1)) (justify left bottom))
-  )
   (text "OK" (at 153.67 33.02 0)
     (effects (font (size 2 2) (color 23 135 61 1)) (justify left bottom))
   )
+  (text "OK" (at 154.94 220.98 0)
+    (effects (font (size 2 2) (color 23 135 61 1)) (justify left bottom))
+  )
   (text "OK" (at 154.94 226.06 0)
     (effects (font (size 2 2) (color 23 135 61 1)) (justify left bottom))
@@
     (effects (font (size 1.27 1.27)) (justify right bottom))
   )
+  (label "IN_VSS" (at 307.34 111.76 180) (fields_autoplaced)
+    (effects (font (size 1.27 1.27)) (justify right bottom))
+  )
   (label "OUT_PUMP_RELAY" (at 307.34 86.36 180) (fields_autoplaced)
     (effects (font (size 1.27 1.27)) (justify right bottom))
@@
     (effects (font (size 1.27 1.27)) (justify left bottom))
   )
+  (label "IN_TEMP" (at 307.34 149.86 180) (fields_autoplaced)
+    (effects (font (size 1.27 1.27)) (justify right bottom))
+  )
+  (label "IN_PPS" (at 307.34 162.56 180) (fields_autoplaced)
+    (effects (font (size 1.27 1.27)) (justify right bottom))
+  )
   (label "IN_IAT" (at 307.34 185.42 180) (fields_autoplaced)
     (effects (font (size 1.27 1.27)) (justify right bottom))
@@
     (effects (font (size 1.27 1.27)) (justify right bottom))
   )
+  (label "IN_O2S" (at 307.34 101.6 180) (fields_autoplaced)
+    (effects (font (size 1.27 1.27)) (justify right bottom))
+  )
   (label "1B" (at 97.79 55.88 180) (fields_autoplaced)
     (effects (font (size 1.27 1.27)) (justify right bottom))
@@
     (effects (font (size 1.27 1.27)) (justify right bottom))
   )
+  (label "OUT_TACH" (at 307.34 71.12 180) (fields_autoplaced)
+    (effects (font (size 1.27 1.27)) (justify right bottom))
+  )
