File: uaefi-adapter-NA6.kicad_sch (KiCad schematic)
At the start: 50 parts, among them P1 178780-1, P10 Pad, P11 Pad, P12 Pad, P2 Pad, P3 Pad, P4 Pad, P5 Pad, P6 Pad, P7 Pad, P8 Pad, P9 Pad

Commit message: upd
Parts:
- removed R18: Jumper-Pad-Pad, hellen-one-common:PAD-0805-PAD, symbol hellen-one-common:Jumper-Pad-Pad
- added P6: Pad, hellen-one-common:PAD-TH, symbol hellen-one-common:Pad
- renumbered F1 to F32, P9 to P10, P7 to P11, P10 to P19, P6 to P2, P8 to P21, P12 to P5, P3 to P55, P2 to P56, P5 to P60, P4 to P63, P11 to P8
Connections:
- net at P1.6 (1K): now also P6.1 (Pin_1)
- no-connect marks 1 -> 0
Other:
- note removed: "!!!!"
- note removed: "OK"
- moved on the sheet: F2, F3, P10, P11, P19, P21, P5, P55, P56, P63, P8, R10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

Commit message: upd
Parts:
- removed BRD?: uaefi, uaefi_brd:UAEFI_BRD, symbol uaefi_brd:UAEFI_BRD
- added J1: 43045-0612, Connector_Molex:Molex_Micro-Fit_3.0_43045-0612_2x03_P3.00mm_Vertical, symbol Connector_Generic:Conn_02x03_Top_Bottom
- added M1: Module:uaefi/0.2, hellen-one-uaefi-0.2:uaefi, symbol hellen-one-uaefi-0.2:Module-uaefi-0.2
- added P3, P4, P7, P9: Pad, kicad6-libraries:PAD-TH, symbol misc:Pad
Connections:
- net +12V_RAW: now also M1.A7 (IN_VIGN), M1.A8 (IN_V_MAIN)
- net GND: now also M1.A3 (GND), M1.A4 (GND), M1.C8 (GND), M1.J4 (GND), M1.J5 (GND)
- net GNDA: now also M1.C11 (GNDA), M1.C12 (GNDA), M1.C13 (GNDA)
- net IN_CAM: now also M1.C5 (IN_HALL1)
- net IN_CLT: now also M1.D16 (IN_CLT)
- net IN_CRANK: now also M1.C7 (IN_HALL3)
- net IN_IAT: now also M1.D15 (IN_IAT)
- net IN_KNOCK_RAW: now also M1.D14 (IN_KNOCK_RAW)
- net IN_TPS: no longer R4.1, R5.1
- net IN_TPS2: now also M1.C14 (IN_TPS2)
- net IN_VSS: now also M1.C6 (IN_HALL2)
- net OUT_AC_RELAY: now also M1.B17 (OUT_LS3)
- net OUT_IDLE: now also M1.B18 (OUT_LS2)
- net OUT_IGN1: now also M1.B15 (OUT_IGN1)
- net OUT_IGN2: now also M1.B14 (OUT_IGN2)
- net OUT_INJ1: now also M1.B6 (OUT_INJ1)
- net OUT_INJ2: now also M1.B5 (OUT_INJ2)
- net OUT_INJ3: now also M1.B4 (OUT_INJ3)
- net OUT_INJ4: now also M1.B3 (OUT_INJ4)
- net OUT_TACH: now also M1.B13 (OUT_IGN5)
- net WBO_Ip: now also M1.E5 (WBO_Ip)
- net WBO_Vs: now also M1.E4 (WBO_Un)
- new net: J1.1 (Pin_1), M1.P4 (LED_GREEN)
- new net: J1.2 (Pin_2), M1.P7 (Rx)
- new net: J1.4 (Pin_4), M1.P3 (LED_YELLOW)
- new net: J1.5 (Pin_5), M1.P8 (Tx)
- new net: M1.P15 (DC1_DIR), P3.1 (Pin_1)
- new net: M1.P16 (DC2_DIR), P7.1 (Pin_1)
- new net: M1.P17 (DC1_PWM), P4.1 (Pin_1)
- new net: M1.P18 (DC2_PWM), P9.1 (Pin_1)
- new net +5VP: M1.C1 (+5VP), M1.C2 (+5VP)
- new net CANH: J1.3 (Pin_3), M1.D7 (CAN+)
- new net CANL: J1.6 (Pin_6), M1.D8 (CAN-)
- new net CKP_24+: M1.C16 (VR_MAX9924+)
- new net CKP_24-: M1.C17 (VR_MAX9924-)
- new net CYP_1+: M1.C18 (VR_DISCRETE+)
- new net CYP_1-: M1.C19 (VR_DISCRETE-)
- new net DC2+: M1.A6 (OUT_DC2+)
- new net ETB_N: M1.A1 (OUT_DC1-)
- new net ETB_P: M1.A5 (OUT_DC1+)
- new net HS_VTC: M1.B10 (OUT_IGN6)
- new net IN_AC_PRESSURE_SW: M1.C15 (IN_AUX3)
- new net IN_DIAG: M1.C9 (IN_BUTTON3)
- new net IN_EGR/AUX1: M1.D1 (IN_AUX1)
- new net IN_FLEX: M1.D5 (IN_FLEX)
- new net IN_HS_BRAKE: M1.D10 (IN_BUTTON2)
- new net IN_HS_START: M1.D2 (IN_BUTTON1)
- new net IN_MAP: M1.D9 (IN_MAP)
- new net IN_O2/AUX2: M1.C3 (IN_AUX2)
- new net IN_PPS1: M1.D6 (IN_PPS1)
- new net IN_PPS2: M1.C4 (IN_PPS2)
- new net IN_TPS1: M1.D13 (IN_TPS1), R4.1, R5.1
- new net OUT_EGR_SOLENOID: M1.B2 (OUT_INJ5)
- new net OUT_FAN_CONTROL: M1.B8 (OUT_LS_WEAK2)
- new net OUT_FUEL_PUMP_RELAY: M1.B16 (OUT_LS4)
- new net OUT_IAB_SOLENOID: M1.B1 (OUT_INJ6)
- new net OUT_IGN3: M1.B12 (OUT_IGN3)
- new net OUT_IGN4: M1.B11 (OUT_IGN4)
- new net OUT_IGNITION_CONTROL_MODULE: M1.B9 (OUT_LS_WEAK1)
- new net OUT_MIL: M1.B7 (OUT_LS1)
- new net WBO_HTR+: M1.E1 (+12V_RAW)
- new net WBO_HTR-: M1.E3 (WBO_Heater)
- new net WBO_Rtrim: M1.E2 (WBO_Rtrim)
- new net WBO_Vm: M1.E6 (WBO_Vm)
- no-connect marks 0 -> 10
Other:
- note added: "Analog inputs (sensors)"
- note added: "Bus types"
- note added: "DC Motor"
- note added: "Discrete inputs"
- note added: "General purpose bus"
- note added: "Ignition"
- note added: "Injection"
- note added: "LS & HS outputs"
- moved on the sheet: F2, F3, F32, P10, P11, P19, P1A, P1B, P1C, P1D, P2, P21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

Commit message: Upd SCH
Parts:
- removed F3: Fuse-Pad-Pad, hellen-one-common:PAD-1206-PAD, symbol hellen-one-common:Fuse-Pad-Pad
- removed R25, R26, R27: Jumper-Pad-Pad, hellen-one-common:PAD-0805-PAD, symbol hellen-one-common:Jumper-Pad-Pad
- removed R32: 1k, hellen-one-common:R0603, symbol hellen-one-common:Res
- added C17: 100n, hellen-one-common:C0603, symbol hellen-one-common:Cap
- added D55: PSM712-LF, hellen-one-common:SOT-23, symbol hellen-one-common:PSM712
- added D56: B5819W, hellen-one-common:SOD-123, symbol hellen-one-common:1N4148WS
- added P12: Pad, hellen-one-common:PAD-TH, symbol hellen-one-common:Pad
- added Q1: ZXMS6005SGTA, Package_TO_SOT_SMD:SOT-223, symbol Power_Management:AUIPS2041L
- added R47: 220, hellen-one-common:R0805, symbol hellen-one-common:Res
- added R47: 750, hellen-one-common:R0805, symbol hellen-one-common:Res
- P1: footprint hellen-one-common:178780-1 -> kicad6-libraries:178780-1
Connections:
- net +5VAS is gone; now on net +5VP: P1.31 (2B), P1.44 (3K), P1.70 (4K), P1.76 (4L), R15.1
- net 1A is gone; now on net +12V_PERM: P1.1 (1A)
- net CAN+ is gone; now on net CANH: R24.1
- net CAN- is gone; now on net CANL: R22.1
- net ETB_N is gone; now on net OUT_ETB-: M1.A1 (OUT_DC1-)
- net ETB_P is gone; now on net OUT_ETB+: M1.A5 (OUT_DC1+)
- net IN_AC_PRESSURE_SW is gone; now on net IN_O2S: M1.C15 (IN_AUX3)
- net IN_DIAG is gone; now on net IN_AC_SW: M1.C9 (IN_BUTTON3)
- net IN_EGR/AUX1 is gone; now on net IN_TEMP: M1.D1 (IN_AUX1)
- net IN_HS_BRAKE is gone; now on net IN_CLUTCH: M1.D10 (IN_BUTTON2)
- net IN_HS_START is gone; now on net IN_DIGITAL: M1.D2 (IN_BUTTON1)
- net IN_MAP is gone; now on net IN_PRESSURE: M1.D9 (IN_MAP)
- net IN_O2/AUX2 is gone; now on net IN_MAF: M1.C3 (IN_AUX2)
- net IN_PPS is gone; now on net IN_PPS1: R9.1
- net IN_PPS2 is gone; now on net IN_TEMP_OR_PPS2: M1.C4 (IN_PPS2)
- net IN_TPS is gone; now on net IN_TPS1: R8.1
- net OUT_EGR_SOLENOID is gone; now on net OUT_AC_RELAY: M1.B2 (OUT_INJ5)
- net OUT_FAN_CONTROL is gone; now on net OUT_RADIATOR_FAN_RELAY: M1.B8 (OUT_LS_HOT2)
- net OUT_FUEL_PUMP_RELAY is gone; now on net OUT_PUMP_RELAY: M1.B16 (OUT_LS4)
- net OUT_IAB_SOLENOID is gone; now on net OUT_CHECK_ENGINE: M1.B1 (OUT_INJ6)
- net OUT_IGNITION_CONTROL_MODULE is gone; now on net OUT_CONDENSER_FAN: M1.B9 (OUT_LS_HOT1)
- net OUT_MIL is gone; now on net OUT_VVT: M1.B7 (OUT_LS1)
- net WBO_HTR- is gone; now on net WBO_H-: M1.E3 (WBO_Heater)
- net WBO_Rtrim is gone; now on net WBO_R_Trim: M1.E2 (WBO_Rtrim)
- net WBO_Vm is gone; now on net WBO_Vs/Ip: M1.E6 (WBO_Vm)
- net +12V_PERM: now also P12.1 (Pin_1)
- net 1B: no longer F32.2
- net GND: now also C17.1, D55.3, Q1.3 (S)
- net OUT_AC_RELAY: no longer M1.B17 (OUT_LS3)
- net OUT_BOOST_CONTROL: now also M1.B17 (OUT_LS3)
- net OUT_TACH: now also R6.1, Q1.2 (D), R47.2; no longer M1.B13 (OUT_IGN5)
- net +12V_RAW renamed 12V_FROM_MAIN_RELAY
- net 12V_FROM_MAIN_RELAY: now also F32.2, R47.2
- net CKP_24+: no longer names the net of M1.C16 (VR_MAX9924+)
- net CKP_24-: no longer names the net of M1.C17 (VR_MAX9924-)
- net CYP_1+: no longer names the net of M1.C18 (VR_DISCRETE+)
- net CYP_1-: no longer names the net of M1.C19 (VR_DISCRETE-)
- net DC2+: no longer names the net of M1.A6 (OUT_DC2+)
- net HS_VTC: no longer names the net of M1.B10 (OUT_IGN6)
- net IN_FLEX: no longer names the net of M1.D5 (IN_FLEX)
- net OUT_IGN3: no longer names the net of M1.B12 (OUT_IGN3)
- net OUT_IGN4: no longer names the net of M1.B11 (OUT_IGN4)
- net WBO_HTR+: no longer names the net of M1.E1 (+12V_RAW)
- new net: C17.2, D55.1, D56.2 (A), R47.1
- new net: D56.1 (K), R47.1
- new net TACH: M1.B13 (OUT_IGN5), Q1.1 (IN)
- no-connect marks 10 -> 21
Other:
- moved on the sheet: P1A, P1B, P1C, P1D

Commit message: upd
Parts:
- added P_C10, P_C11, P_C12, P_C13, P_C20, P_D5: Pad, hellen-one-common:PAD-TH, symbol hellen-one-common:Pad
Connections:
- net GNDA: now also P_C11.1 (Pin_1), P_C12.1 (Pin_1), P_C13.1 (Pin_1)
- net at M1.C10 (EGT+): now also P_C10.1 (Pin_1)
- net at M1.C20 (EGT-): now also P_C20.1 (Pin_1)
- net at M1.D5 (IN_FLEX): now also P_D5.1 (Pin_1)
Other:
- moved on the sheet: P2, P55

Commit message: upd
Parts:
- added G1, G2, G3, G4, G5, G6, G7: PROTO_AREA_2, hellen-one-common:PROTO_AREA_2, symbol hellen-one-common:PROTO_AREA_2
Connections:
- net GND: now also G1.1, G1.2, G1.6, G1.7
- new net: G1.10, G1.5
- new net: G1.3, G1.8
- new net: G1.4, G1.9
- new net: G7.1, G7.6
- new net: G7.10, G7.5
- new net: G7.2, G7.7
- new net: G7.3, G7.8
- new net: G7.4, G7.9
- new net: G3.1, G3.6
- new net: G3.10, G3.5
- new net: G3.2, G3.7
- new net: G3.3, G3.8
- new net: G3.4, G3.9
- new net: G4.1, G4.6
- new net: G4.10, G4.5
- new net: G4.2, G4.7
- new net: G4.3, G4.8
- new net: G4.4, G4.9
- new net: G5.1, G5.6
- new net: G5.10, G5.5
- new net: G5.2, G5.7
- new net: G5.3, G5.8
- new net: G5.4, G5.9
- new net: G2.1, G2.6
- new net: G2.10, G2.5
- new net: G2.2, G2.7
- new net: G2.3, G2.8
- new net: G2.4, G2.9
- new net: G6.1, G6.6
- new net: G6.10, G6.5
- new net: G6.2, G6.7
- new net: G6.3, G6.8
- new net: G6.4, G6.9
Other:
- note added: "Prototype areas"
- moved on the sheet: C17, D55, D56, F2, F32, J1, M1, P10, P11, P12, P19, P1A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
