File: uaefi-adapter-NA-90-95.kicad_sch (KiCad schematic)
At the start: 70 parts, among them J1 43045-0612, M1 Module:uaefi/0.2, P1 178780-1, P10 Pad, P11 Pad, P12 Pad, P19 Pad, P2 Pad, P21 Pad, P3 Pad, P4 Pad, P5 Pad, P55 Pad, P56 Pad, P6 Pad, P60 Pad, P63 Pad, P7 Pad, P8 Pad, P9 Pad, Q1 ZXMS6005SGTA

Commit message: upd
Parts:
- renumbered F2 to F12, R24 to R13, R22 to R14, R20 to R15, R19 to R16, R15 to R18, R13 to R20, R12 to R22, R23 to R3, R21 to R4, R6 to R43, R4 to R45, R29 to R46, R28 to R46_61, R2 to R48, R34 to R49_51, R31 to R51, R7 to R54, R5 to R57, R3 to R58, R1 to R61, R33 to R62_64, R30 to R64, R11 to R68, R9 to R69, R16 to R7, R10 to R74, R8 to R75, R14 to R9

Commit message: upd
Parts:
- removed G1, G2, G3, G4, G5, G6, G7: PROTO_AREA_2, hellen-one-common:PROTO_AREA_2, symbol hellen-one-common:PROTO_AREA_2
- added G10, G11, G8, G9: PROTO_AREA, hellen-one-common:PROTO_AREA, symbol hellen-one-common:PROTO_AREA
- P1: footprint kicad6-libraries:178780-1 -> 178780-1:178780-1_OBD1
Connections:
- net GND: now also G8.1, G8.11, G8.12, G8.2, G8.6, G8.7

Commit message: upd
Parts:
- added J2: 43045-0412, Connector_Molex:Molex_Micro-Fit_3.0_43045-0412_2x02_P3.00mm_Vertical, symbol Connector_Generic:Conn_02x02_Top_Bottom
Connections:
- net at M1.C16 (VR_MAX9924+): now also J2.1 (Pin_1)
- net at M1.C17 (VR_MAX9924-): now also J2.3 (Pin_3)
- net at M1.C18 (VR_DISCRETE+): now also J2.2 (Pin_2)
- net at M1.C19 (VR_DISCRETE-): now also J2.4 (Pin_4)
- no-connect marks 18 -> 14
Changed lines of the file:
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@@
   (junction (at 229.87 72.39) (diameter 0) (color 0 0 0 0)
   )
-  (no_connect (at 387.35 158.75))
   (no_connect (at 387.35 199.39))
   (no_connect (at 387.35 234.95))
@@
   (no_connect (at 387.35 237.49))
   (no_connect (at 387.35 97.79))
-  (no_connect (at 387.35 161.29))
   (no_connect (at 387.35 214.63))
   (no_connect (at 387.35 92.71))
-  (no_connect (at 387.35 163.83))
   (no_connect (at 387.35 49.53))
-  (no_connect (at 387.35 156.21))
   (no_connect (at 387.35 59.69))
   (no_connect (at 326.39 95.25))
@@
     (stroke (width 0) (type default))
   )
+  (wire (pts (xy 358.14 165.1) (xy 358.14 161.29))
+    (stroke (width 0) (type default))
+  )
   (wire (pts (xy 127 220.98) (xy 294.64 220.98))
     (stroke (width 0) (type solid))
@@
     (stroke (width 0) (type default))
   )
+  (wire (pts (xy 372.11 158.75) (xy 387.35 158.75))
+    (stroke (width 0) (type default))
+  )
   (bus (pts (xy 222.25 250.19) (xy 222.25 247.65))
     (stroke (width 0) (type default) (color 255 0 255 1))
@@
     (stroke (width 0) (type default))
   )
+  (wire (pts (xy 358.14 161.29) (xy 359.41 161.29))
+    (stroke (width 0) (type default))
+  )
   (wire (pts (xy 105.41 106.68) (xy 129.54 106.68))
     (stroke (width 0) (type solid))
@@
     (stroke (width 0) (type solid))
   )
+  (wire (pts (xy 358.14 156.21) (xy 358.14 158.75))
+    (stroke (width 0) (type default))
+  )
   (bus (pts (xy 229.87 142.24) (xy 229.87 182.88))
     (stroke (width 0) (type default) (color 255 153 0 1))
@@
     (stroke (width 0) (type default))
   )
+  (wire (pts (xy 384.81 161.29) (xy 384.81 165.1))
+    (stroke (width 0) (type default))
+  )
   (bus (pts (xy 350.52 59.69) (xy 292.1 59.69))
     (stroke (width 0) (type default) (color 0 194 194 1))
@@
     (stroke (width 0) (type default))
   )
+  (wire (pts (xy 379.73 163.83) (xy 379.73 161.29))
+    (stroke (width 0) (type default))
+  )
   (bus (pts (xy 351.79 92.71) (xy 351.79 110.49))
     (stroke (width 0) (type default) (color 255 153 0 1))
@@
     (stroke (width 0) (type default))
   )
+  (wire (pts (xy 384.81 165.1) (xy 358.14 165.1))
+    (stroke (width 0) (type default))
+  )
   (wire (pts (xy 105.41 185.42) (xy 190.5 185.42))
     (stroke (width 0) (type solid))
@@
     (stroke (width 0) (type solid))
   )
+  (wire (pts (xy 358.14 158.75) (xy 359.41 158.75))
+    (stroke (width 0) (type default))
+  )
   (wire (pts (xy 105.41 77.47) (xy 116.84 77.47))
     (stroke (width 0) (type solid))
@@
     (stroke (width 0) (type default) (color 255 153 0 1))
   )
+  (wire (pts (xy 387.35 163.83) (xy 379.73 163.83))
+    (stroke (width 0) (type default))
+  )
   (bus (pts (xy 350.52 135.89) (xy 350.52 140.97))
     (stroke (width 0) (type default) (color 194 194 0 1))
@@
     (stroke (width 0) (type default) (color 255 0 0 1))
   )
+  (wire (pts (xy 387.35 161.29) (xy 384.81 161.29))
+    (stroke (width 0) (type default))
+  )
   (wire (pts (xy 144.78 116.84) (xy 140.97 116.84))
     (stroke (width 0) (type solid))
@@
     (stroke (width 0) (type default))
   )
+  (wire (pts (xy 372.11 161.29) (xy 379.73 161.29))
+    (stroke (width 0) (type default))
+  )
   (wire (pts (xy 353.06 57.15) (xy 387.35 57.15))
     (stroke (width 0) (type default))
   )
+  (wire (pts (xy 387.35 156.21) (xy 358.14 156.21))
+    (stroke (width 0) (type default))
+  )
   (wire (pts (xy 158.75 111.76) (xy 219.71 111.76))
     (stroke (width 0) (type default))
@@
         )
       )
+    )
+  )
+  (symbol (lib_id "Connector_Generic:Conn_02x02_Top_Bottom") (at 364.49 158.75 0) (unit 1)
+    (in_bom yes) (on_board yes) (dnp no)
+    (property "Reference" "J2" (at 365.7606 155.2228 0)
+      (effects (font (size 1.27 1.27)))
+    )
+    (property "Value" "43045-0412" (at 365.6404 163.6469 0)
+      (effects (font (size 1.27 1.27)))
+    )
+    (property "Footprint" "Connector_Molex:Molex_Micro-Fit_3.0_43045-0412_2x02_P3.00mm_Vertical" (at 364.49 158.75 0)
+      (effects (font (size 1.27 1.27)) hide)
+    )
+    (property "Datasheet" "~" (at 364.49 158.75 0)
+      (effects (font (size 1.27 1.27)) hide)
+    )
+    (pin "1")
+    (pin "2")
+    (pin "3")
+    (pin "4")
+    (instances
+      (project "uaefi-adapter-NA-90-95"
+        (path "/62be380c-4f45-483a-9614-39f0039d587a"
+          (reference "J2") (unit 1)
+        )
+      )
