File: uaefi-adapter-NA-90-95.kicad_sch (KiCad schematic)
At the start: 68 parts, among them J1 43045-0612, J2 43045-0412, M1 Module:uaefi/0.2, P1 178780-1, P10 Pad, P11 Pad, P12 Pad, P19 Pad, P2 Pad, P21 Pad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

Commit message: upd
Parts:
- removed P_C10, P_C20: Pad, hellen-one-common:PAD-TH, symbol hellen-one-common:Pad
- added J3: 43045-0212, Connector_Molex:Molex_Micro-Fit_3.0_43045-0212_2x01_P3.00mm_Vertical, symbol Connector_Generic:Conn_02x01
Connections:
- net +5VP: now also G8.13, G8.14, G8.3, G8.4, G8.8, G8.9
- net 12V_FROM_MAIN_RELAY: now also G8.10, G8.15, G8.5
- net GNDA: no longer M1.C11 (GNDA), M1.C12 (GNDA), M1.C13 (GNDA), P_C11.1 (Pin_1), P_C12.1 (Pin_1), P_C13.1 (Pin_1)
- new net: M1.C12 (GNDA), P_C12.1 (Pin_1)
- new net: M1.C11 (GNDA), P_C11.1 (Pin_1)
- new net: M1.C13 (GNDA), P_C13.1 (Pin_1)
- new net EGT+: J3.1 (Pin_1)
- new net EGT-: J3.2 (Pin_2)
Other:
- moved on the sheet: P_C11, P_C12, P_C13, P_D5

Commit message: upd
Connections:
- net EGT+: now also M1.C10 (EGT+)
- net EGT-: now also M1.C20 (EGT-)
Changed lines of the file:
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@@
     (effects (font (size 1.27 1.27)) (justify right bottom))
+  )
+  (label "EGT-" (at 353.06 166.37 0) (fields_autoplaced)
+    (effects (font (size 1.27 1.27)) (justify left bottom))
   )
   (label "IN_TEMP_OR_PPS2" (at 190.5 247.65 180) (fields_autoplaced)
@@
     (effects (font (size 1.27 1.27)) (justify right bottom))
   )
+  (label "EGT+" (at 358.14 140.97 180) (fields_autoplaced)
+    (effects (font (size 1.27 1.27)) (justify right bottom))
+  )

Commit message: upd
Connections:
- net GNDA: now also M1.C11 (GNDA), M1.C12 (GNDA), M1.C13 (GNDA), P_C11.1 (Pin_1), P_C12.1 (Pin_1), P_C13.1 (Pin_1)
Changed lines of the file:
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@@
+    (effects (font (size 1.27 1.27)) (justify left bottom))
+  )
+  (label "GNDA" (at 373.38 146.05 0) (fields_autoplaced)
     (effects (font (size 1.27 1.27)) (justify left bottom))
   )
@@
     (effects (font (size 1.27 1.27)) (justify left bottom))
   )
+  (label "GNDA" (at 373.38 143.51 0) (fields_autoplaced)
+    (effects (font (size 1.27 1.27)) (justify left bottom))
+  )
   (label "OUT_PUMP_RELAY" (at 354.33 107.95 0) (fields_autoplaced)
     (effects (font (size 1.27 1.27)) (justify left bottom))
@@
     (effects (font (size 1.27 1.27)) (justify left bottom))
   )
+  (label "GNDA" (at 373.38 148.59 0) (fields_autoplaced)
+    (effects (font (size 1.27 1.27)) (justify left bottom))
+  )
