File: uaefi-adapter-NA-90-95.kicad_pcb (KiCad board)
At the start: 2 copper layers, 154 x 159 mm, 58 parts, among them J1 43045-0612, J11 Conn_01x01, J13 Conn_01x01, J14 Conn_01x01, J15 Conn_01x01, J16 Conn_01x01, J17 Conn_01x01, P10 Pad, P15 Pad, P16 Pad, P17 Pad, P19 Pad, P2 Pad, P21 Pad, P3 Pad, P46 Pad, P7 Pad, P8 Pad, P9 Pad, Q1 ZXMS6005SGTA

Commit message: upd
Parts:
- removed BRD1: uaefi, uaefi_brd:UAEFI_BRD
- removed F1, F2, F3: Fuse-Pad-Pad, hellen-one-common:PAD-1206-PAD
- removed P15, P16, P17, P46: Pad, hellen-one-common:PAD-TH
- removed R12, R19, R24, R26, R27, R28, R30, R31, R32, R33, R34, R35, R36, R37, R38, R39, R40, R42, R44, R47, R49, R52, R8: Jumper-Pad-Pad, hellen-one-common:PAD-0805-PAD
- removed R21: Jumper-Pad-Pad, hellen-one-common:R0603
- added C1: 100n, hellen-one-common:C0603, F.Cu at (206.9, 71.3)
- added D1: B5819W, hellen-one-common:SOD-123, F.Cu at (222.3, 73.7)
- added D2: PSM712-LF, hellen-one-common:SOT-23, F.Cu at (202.7, 72.6)
- added F12: Fuse-Pad-Pad, hellen-one-common:PAD-1206-PAD, F.Cu at (223.5, 67.5)
- added F32: Fuse-Pad-Pad, hellen-one-common:PAD-1206-PAD, F.Cu at (223.5, 70.6)
- added G10: PROTO_AREA, hellen-one-common:PROTO_AREA, F.Cu at (197.9, 55.5)
- added G11: PROTO_AREA, hellen-one-common:PROTO_AREA, F.Cu at (197.9, 63.7)
- added G8: PROTO_AREA, hellen-one-common:PROTO_AREA, F.Cu at (197.9, 39.0)
- added G9: PROTO_AREA, hellen-one-common:PROTO_AREA, F.Cu at (197.9, 47.2)
- added M1: Module:uaefi/0.2, hellen-one-uaefi-0.2:uaefi, F.Cu at (46.0, 170.5)
- added P11: Pad, hellen-one-common:PAD-TH, F.Cu at (235.3, 50.6)
- added P12: Pad, hellen-one-common:PAD-TH, F.Cu at (235.3, 54.4)
- added P2: Pad, hellen-one-common:PAD-TH, F.Cu at (231.5, 39.3)
- added P4: Pad, kicad6-libraries:PAD-TH, F.Cu at (231.5, 46.9)
- added P5: Pad, hellen-one-common:PAD-TH, F.Cu at (231.5, 50.6)
- added P55: Pad, hellen-one-common:PAD-TH, F.Cu at (239.1, 43.1)
- added P56: Pad, hellen-one-common:PAD-TH, F.Cu at (239.1, 46.9)
- added P6: Pad, hellen-one-common:PAD-TH, F.Cu at (231.5, 54.4)
- added P60: Pad, hellen-one-common:PAD-TH, F.Cu at (239.1, 50.6)
- added P63: Pad, hellen-one-common:PAD-TH, F.Cu at (239.1, 54.4)
- added P_C10: Pad, hellen-one-common:PAD-TH, F.Cu at (239.1, 58.2)
- added P_C11: Pad, hellen-one-common:PAD-TH, F.Cu at (242.9, 39.3)
- added P_C12: Pad, hellen-one-common:PAD-TH, F.Cu at (242.9, 43.1)
- added P_C13: Pad, hellen-one-common:PAD-TH, F.Cu at (242.9, 46.9)
- added P_C20: Pad, hellen-one-common:PAD-TH, F.Cu at (242.9, 50.6)
- added P_D5: Pad, hellen-one-common:PAD-TH, F.Cu at (242.9, 54.4)
- added R1: 750, hellen-one-common:R0805, F.Cu at (198.3, 71.6)
- added R13: Jumper-Pad-Pad, hellen-one-common:PAD-0805-PAD, F.Cu at (213.0, 50.2)
- added R14: Jumper-Pad-Pad, hellen-one-common:PAD-0805-PAD, F.Cu at (213.0, 53.1)
- added R15: Jumper-Pad-Pad, hellen-one-common:PAD-0805-PAD, F.Cu at (213.0, 55.9)
- added R16: Jumper-Pad-Pad, hellen-one-common:PAD-0805-PAD, F.Cu at (213.0, 58.8)
- added R20: Jumper-Pad-Pad, hellen-one-common:PAD-0805-PAD, F.Cu at (219.7, 38.8)
- added R3: Jumper-Pad-Pad, hellen-one-common:PAD-0805-PAD, F.Cu at (213.0, 38.8)
- added R4: Jumper-Pad-Pad, hellen-one-common:PAD-0805-PAD, F.Cu at (213.0, 41.7)
- added R46_61: Jumper-Pad-Pad, hellen-one-common:PAD-0805-PAD, F.Cu at (226.3, 55.9)
- added R49_51: Jumper-Pad-Pad, hellen-one-common:PAD-0805-PAD, F.Cu at (226.3, 58.8)
- added R54: Jumper-Pad-Pad, hellen-one-common:PAD-0805-PAD, F.Cu at (219.7, 58.8)
- added R57: Jumper-Pad-Pad, hellen-one-common:PAD-0805-PAD, F.Cu at (219.7, 61.6)
- added R61: Jumper-Pad-Pad, hellen-one-common:PAD-0805-PAD, F.Cu at (226.3, 38.8)
- added R62_64: Jumper-Pad-Pad, hellen-one-common:PAD-0805-PAD, F.Cu at (226.3, 61.6)
- added R64: Jumper-Pad-Pad, hellen-one-common:PAD-0805-PAD, F.Cu at (226.3, 41.7)
- added R68: Jumper-Pad-Pad, hellen-one-common:PAD-0805-PAD, F.Cu at (226.3, 44.5)
- added R69: Jumper-Pad-Pad, hellen-one-common:PAD-0805-PAD, F.Cu at (226.3, 47.4)
- added R7: Jumper-Pad-Pad, hellen-one-common:PAD-0805-PAD, F.Cu at (213.0, 44.5)
- added R74: Jumper-Pad-Pad, hellen-one-common:PAD-0805-PAD, F.Cu at (226.3, 50.2)
- added R75: Jumper-Pad-Pad, hellen-one-common:PAD-0805-PAD, F.Cu at (226.3, 53.1)
- added R9: Jumper-Pad-Pad, hellen-one-common:PAD-0805-PAD, F.Cu at (213.0, 47.4)
- P1: renamed from P2; value Pad -> 178780-1
- P3, P7, P9: footprint hellen-one-common:PAD-TH -> kicad6-libraries:PAD-TH
- R18: value 750 -> Jumper-Pad-Pad
- R25: footprint hellen-one-common:PAD-0805-PAD -> hellen-one-common:R0805
- moved P10 190.5 mm to (235.3, 46.9), turned to 0 degrees
- moved P21 182.8 mm to (239.1, 39.3), turned to 0 degrees
- moved P19 178.5 mm to (235.3, 58.2)
- moved R58 156.7 mm to (219.7, 64.5), turned to 0 degrees
- moved R51 138.8 mm to (219.7, 55.9), turned to 0 degrees
- moved R22 136.6 mm to (219.7, 41.7), turned to 0 degrees
- moved P7 103.6 mm to (231.5, 58.2), turned to 0 degrees
- moved P3 103.5 mm to (231.5, 43.1)
- moved P9 92.5 mm to (235.3, 43.1), turned to 0 degrees
- moved R48 86.8 mm to (219.7, 53.1), turned to 0 degrees
- moved P8 83.7 mm to (235.3, 39.3)
- moved R46 82.2 mm to (219.7, 50.2), turned to 0 degrees
- moved R45 74.9 mm to (219.7, 47.4), turned to 0 degrees
- moved R43 72.9 mm to (219.7, 44.5), turned to 0 degrees
- moved R18 70.3 mm to (213.0, 64.5), turned to 0 degrees
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Connections:
- P1 pad 1: /1C -> /+12V_PERM
- P1 pad 10: (no net) -> Net-(P10-Pin_1)
- P1 pad 11: (no net) -> /1U
- P1 pad 12: (no net) -> /1B
- P1 pad 13: (no net) -> /1D
- P1 pad 14: (no net) -> /1F
- P1 pad 15: (no net) -> /1H
- P1 pad 16: (no net) -> /1J
- P1 pad 17: (no net) -> /1L
- P1 pad 18: (no net) -> /1N
- P1 pad 19: (no net) -> /1P
- P1 pad 2: (no net) -> /1C
- P1 pad 20: (no net) -> Net-(P1A-1R)
- P1 pad 21: (no net) -> Net-(P1A-1T)
- P1 pad 22: (no net) -> /1V
- P1 pad 23: (no net) -> GND
- P1 pad 24: (no net) -> /WBO_H-
- P1 pad 25: (no net) -> /WBO_R_Trim
- P1 pad 26: (no net) -> /WBO_Vs/Ip
- P1 pad 27: (no net) -> /OUT_VVT
- P1 pad 28: (no net) -> GND
- P1 pad 29: (no net) -> /IN_PRESSURE
- P1 pad 3: (no net) -> /1E
- P1 pad 30: (no net) -> GND
- P1 pad 31: (no net) -> +5VP
- P1 pad 32: (no net) -> /2D
- P1 pad 33: (no net) -> /WBO_Ip
- P1 pad 34: (no net) -> /WBO_Vs
- P1 pad 35: (no net) -> /OUT_BOOST_CONTROL
- P1 pad 36: (no net) -> /IN_DIGITAL
- P1 pad 37: (no net) -> /IN_TEMP
- P1 pad 38: (no net) -> /IN_KNOCK_RAW
- P1 pad 39: (no net) -> GND
- P1 pad 4: (no net) -> /1G
- P1 pad 40: (no net) -> GNDA
- P1 pad 41: (no net) -> /IN_CRANK
- P1 pad 42: (no net) -> /IN_CAM
- P1 pad 43: (no net) -> /3I
- P1 pad 44: (no net) -> +5VP
- P1 pad 45: (no net) -> /3M
- P1 pad 46: (no net) -> /3O
- P1 pad 47: (no net) -> /IN_CLT
- P1 pad 48: (no net) -> /3S
- P1 pad 49: (no net) -> /OUT_INJ1
- P1 pad 5: (no net) -> Net-(P1A-1I)
- P1 pad 50: (no net) -> /OUT_IDLE
- P1 pad 51: (no net) -> /3Y
- P1 pad 52: (no net) -> GNDA
- P1 pad 53: (no net) -> GNDA
- P1 pad 54: (no net) -> /3F
- P1 pad 55: (no net) -> /3H
- P1 pad 56: (no net) -> /3J
- P1 pad 57: (no net) -> /3L
- P1 pad 58: (no net) -> /3N
- P1 pad 59: (no net) -> /IN_IAT
- P1 pad 6: (no net) -> Net-(P1A-1K)
- P1 pad 60: (no net) -> /3R
- P1 pad 61: (no net) -> /3T
- P1 pad 62: (no net) -> /OUT_INJ2
- P1 pad 63: (no net) -> /3X
- P1 pad 64: (no net) -> /3Z
- P1 pad 65: (no net) -> /OUT_ETB+
- P1 pad 66: (no net) -> /OUT_ETB-
- P1 pad 67: (no net) -> GNDA
- P1 pad 68: (no net) -> Net-(P1D-4G)
- P1 pad 69: (no net) -> Net-(P1D-4I)
- P1 pad 7: (no net) -> /1M
- P1 pad 70: (no net) -> +5VP
- P1 pad 71: (no net) -> /OUT_ETB+
- P1 pad 72: (no net) -> /OUT_ETB-
- P1 pad 73: (no net) -> GNDA
- P1 pad 74: (no net) -> Net-(P1D-4H)
- P1 pad 75: (no net) -> Net-(P1D-4J)
- P1 pad 76: (no net) -> +5VP
- P1 pad 8: (no net) -> /1O
- P1 pad 9: (no net) -> /1Q
- R18 pad 1: Net-(D1-K) -> +5VP
- R18 pad 2: /OUT_TACH -> /1N
- R22 pad 1: /CANL -> /IN_CLUTCH
- R22 pad 2: /1F -> /1V
- R43 pad 1: (no net) -> /OUT_TACH
- R43 pad 2: (no net) -> /3I
- R45 pad 1: (no net) -> /IN_TPS1
- R45 pad 2: (no net) -> /3M
- R46 pad 1: (no net) -> /IN_MAF
- R46 pad 2: (no net) -> /3O
- R48 pad 1: (no net) -> /OUT_CONDENSER_FAN
- R48 pad 2: (no net) -> /3S
- R51 pad 1: (no net) -> /OUT_INJ3
- R51 pad 2: (no net) -> /3Y
- R58 pad 1: (no net) -> /IN_O2S
- R58 pad 2: (no net) -> /3N
Routing:
- net (no net): track 873.9 -> 0.00 mm, vias 7 -> 0
- net /1B: track 77.4 -> 0.00 mm
- net /OUT_INJ3: track 76.4 -> 0.00 mm, vias 1 -> 0
- net /12V_FROM_MAIN_RELAY: track 31.6 -> 0.00 mm
- net /1L: track 25.8 -> 0.00 mm
- net Net-(P1D-4J): track 24.8 -> 0.00 mm
- net Net-(P10-Pin_1): track 22.8 -> 0.00 mm
- net /1V: track 21.2 -> 0.00 mm
- net Net-(P1A-1T): track 19.4 -> 0.00 mm
- net /OUT_TACH: track 16.3 -> 0.00 mm
- net Net-(M1-DC1_DIR): track 15.6 -> 0.00 mm
- net /1O: track 15.1 -> 0.00 mm
- net /3O: track 14.9 -> 0.00 mm
- net Net-(M1-DC2_PWM): track 13.8 -> 0.00 mm
- net /3Y: track 12.4 -> 0.00 mm
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Other:
- outline, holes or cut-outs redrawn
- board text removed: "PRESSURE"

Commit message: upd
Parts:
- added J2: 43045-0412, Connector_Molex:Molex_Micro-Fit_3.0_43045-0412_2x02_P3.00mm_Vertical, F.Cu at (250.5, 62.6)
Connections:
- M1 pad C16: unconnected-(M1-VR_MAX9924+-PadC16) -> Net-(J2-Pin_1)
- M1 pad C17: unconnected-(M1-VR_MAX9924--PadC17) -> Net-(J2-Pin_3)
- M1 pad C18: unconnected-(M1-VR_DISCRETE+-PadC18) -> Net-(J2-Pin_2)
- M1 pad C19: unconnected-(M1-VR_DISCRETE--PadC19) -> Net-(J2-Pin_4)
Changed lines of the file:
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@@
   (net 120 "/IN_TPS2")
   (net 121 "/IN_O2S")
-  (net 122 "unconnected-(M1-VR_MAX9924+-PadC16)")
-  (net 123 "unconnected-(M1-VR_MAX9924--PadC17)")
-  (net 124 "unconnected-(M1-VR_DISCRETE+-PadC18)")
-  (net 125 "unconnected-(M1-VR_DISCRETE--PadC19)")
+  (net 122 "Net-(J2-Pin_1)")
+  (net 123 "Net-(J2-Pin_2)")
+  (net 124 "Net-(J2-Pin_3)")
+  (net 125 "Net-(J2-Pin_4)")
   (net 126 "Net-(M1-EGT-)")
   (net 127 "/IN_TEMP")
@@
     )
   )
+  (footprint "Connector_Molex:Molex_Micro-Fit_3.0_43045-0412_2x02_P3.00mm_Vertical" (layer "F.Cu")
+    (at 250.5 62.585)
+    (descr "Molex Micro-Fit 3.0 Connector System, 43045-0412 (compatible alternatives: 43045-0413, 43045-0424), 2 Pins per row (http://www.molex.com/pdm_docs/sd/430450212_sd.pdf), generated with kicad-footprint-generator")
+    (tags "connector Molex Micro-Fit_3.0 side entry")
+    (property "Sheetfile" "uaefi-adapter-NA-90-95.kicad_sch")
+    (property "Sheetname" "")
+    (property "ki_description" "Generic connector, double row, 02x02, top/bottom pin numbering scheme (row 1: 1...pins_per_row, row2: pins_per_row+1 ... num_pins), script generated (kicad-library-utils/schlib/autogen/connector/)")
+    (property "ki_keywords" "connector")
+    (attr through_hole)
+    (fp_text reference "J2" (at 1.5 -3.67) (layer "F.SilkS")
+        (effects (font (size 1 1) (thickness 0.15)))
+    )
+    (fp_text value "43045-0412" (at 1.5 7.5) (layer "F.Fab")
+        (effects (font (size 1 1) (thickness 0.15)))
+    )
+    (fp_text user "${REFERENCE}" (at 1.5 4.2) (layer "F.Fab")
+        (effects (font (size 1 1) (thickness 0.15)))
+    )
+    (fp_line (start -3.435 -2.58) (end -2.015 -2.58)
+      (stroke (width 0.12) (type solid)) (layer "F.SilkS"))
+    (fp_line (start -3.435 3.18) (end -3.435 -2.58)
+      (stroke (width 0.12) (type solid)) (layer "F.SilkS"))
+    (fp_line (start -3.435 4.7) (end -3.435 5.01)
+      (stroke (width 0.12) (type solid)) (layer "F.SilkS"))
+    (fp_line (start -3.435 5.01) (end 6.435 5.01)
+      (stroke (width 0.12) (type solid)) (layer "F.SilkS"))
+    (fp_line (start -2.015 -2.58) (end -2.015 -2.08)
+      (stroke (width 0.12) (type solid)) (layer "F.SilkS"))
+    (fp_line (start -2.015 -2.08) (end 5.015 -2.08)
+      (stroke (width 0.12) (type solid)) (layer "F.SilkS"))
+    (fp_line (start 5.015 -2.58) (end 6.435 -2.58)
+      (stroke (width 0.12) (type solid)) (layer "F.SilkS"))
+    (fp_line (start 5.015 -2.08) (end 5.015 -2.58)
+      (stroke (width 0.12) (type solid)) (layer "F.SilkS"))
+    (fp_line (start 6.435 -2.58) (end 6.435 3.18)
+      (stroke (width 0.12) (type solid)) (layer "F.SilkS"))
+    (fp_line (start 6.435 5.01) (end 6.435 4.7)
+      (stroke (width 0.12) (type solid)) (layer "F.SilkS"))
+    (fp_line (start -3.82 -2.97) (end 6.82 -2.97)
+      (stroke (width 0.05) (type solid)) (layer "F.CrtYd"))
+    (fp_line (start -3.82 6.8) (end -3.82 -2.97)
+      (stroke (width 0.05) (type solid)) (layer "F.CrtYd"))
+    (fp_line (start 6.82 -2.97) (end 6.82 6.8)
+      (stroke (width 0.05) (type solid)) (layer "F.CrtYd"))
+    (fp_line (start 6.82 6.8) (end -3.82 6.8)
+      (stroke (width 0.05) (type solid)) (layer "F.CrtYd"))
+    (fp_line (start -3.325 -2.47) (end -3.325 4.9)
+      (stroke (width 0.1) (type solid)) (layer "F.Fab"))
+    (fp_line (start -3.325 -1.34) (end -2.125 -1.97)
+      (stroke (width 0.1) (type solid)) (layer "F.Fab"))
+    (fp_line (start -3.325 4.9) (end 6.325 4.9)
+      (stroke (width 0.1) (type solid)) (layer "F.Fab"))
+    (fp_line (start -2.125 -2.47) (end -3.325 -2.47)
+      (stroke (width 0.1) (type solid)) (layer "F.Fab"))
+    (fp_line (start -2.125 -1.97) (end -2.125 -2.47)
+      (stroke (width 0.1) (type solid)) (layer "F.Fab"))
+    (fp_line (start -0.5 -1.97) (end 0 -1.262893)
+      (stroke (width 0.1) (type solid)) (layer "F.Fab"))
+    (fp_line (start 0 -1.262893) (end 0.5 -1.97)
+      (stroke (width 0.1) (type solid)) (layer "F.Fab"))
+    (fp_line (start 0.8 4.9) (end 0.8 6.3)
+      (stroke (width 0.1) (type solid)) (layer "F.Fab"))
+    (fp_line (start 0.8 6.3) (end 2.2 6.3)
+      (stroke (width 0.1) (type solid)) (layer "F.Fab"))
+    (fp_line (start 2.2 6.3) (end 2.2 4.9)
+      (stroke (width 0.1) (type solid)) (layer "F.Fab"))
+    (fp_line (start 5.125 -2.47) (end 5.125 -1.97)
+      (stroke (width 0.1) (type solid)) (layer "F.Fab"))
+    (fp_line (start 5.125 -1.97) (end -2.125 -1.97)
+      (stroke (width 0.1) (type solid)) (layer "F.Fab"))
+    (fp_line (start 6.325 -2.47) (end 5.125 -2.47)
+      (stroke (width 0.1) (type solid)) (layer "F.Fab"))
+    (fp_line (start 6.325 -1.34) (end 5.125 -1.97)
+      (stroke (width 0.1) (type solid)) (layer "F.Fab"))
+    (fp_line (start 6.325 4.9) (end 6.325 -2.47)
+      (stroke (width 0.1) (type solid)) (layer "F.Fab"))
+    (pad "" np_thru_hole circle (at -3 3.94) (size 1 1) (drill 1) (layers "*.Cu" "*.Mask"))
+    (pad "" np_thru_hole circle (at 6 3.94) (size 1 1) (drill 1) (layers "*.Cu" "*.Mask"))
+    (pad "1" thru_hole roundrect (at 0 0) (size 1.5 1.5) (drill 1) (layers "*.Cu" "*.Mask") (roundrect_rratio 0.166667)
+      (net 122 "Net-(J2-Pin_1)") (pinfunction "Pin_1") (pintype "passive"))
+    (pad "2" thru_hole circle (at 3 0) (size 1.5 1.5) (drill 1) (layers "*.Cu" "*.Mask")
+      (net 123 "Net-(J2-Pin_2)") (pinfunction "Pin_2") (pintype "passive"))
+    (pad "3" thru_hole circle (at 0 3) (size 1.5 1.5) (drill 1) (layers "*.Cu" "*.Mask")
+      (net 124 "Net-(J2-Pin_3)") (pinfunction "Pin_3") (pintype "passive"))
+    (pad "4" thru_hole circle (at 3 3) (size 1.5 1.5) (drill 1) (layers "*.Cu" "*.Mask")
+      (net 125 "Net-(J2-Pin_4)") (pinfunction "Pin_4") (pintype "passive"))
+    (model "${KICAD6_3DMODEL_DIR}/Connector_Molex.3dshapes/Molex_Micro-Fit_3.0_43045-0412_2x02_P3.00mm_Vertical.wrl"
+      (offset (xyz 0 0 0))
+      (scale (xyz 1 1 1))
+      (rotate (xyz 0 0 0))
+    )
+  )
   (footprint "hellen-one-common:PAD-0805-PAD" placed (layer "F.Cu")
     (at 226.326953 55.940083)
@@
     (fp_arc (start 23 -13) (mid 24.414214 -12.414214) (end 25 -11)
       (stroke (width 0.1) (type default)) (layer "Edge.Cuts"))
-    (fp_arc (start 27 -1.287437) (mid 25.5858 -1.873226) (end 25 -3.287437)
+    (fp_arc (start 27 -1.287437) (mid 25.585764 -1.87322) (end 25 -3.287437)
       (stroke (width 0.1) (type default)) (layer "Edge.Cuts"))
     (fp_arc (start 59.899911 -8.00008) (mid 60.48572 -9.414273) (end 61.899911 -10.00008)
@@
     (fp_arc (start 59.9 -3.3) (mid 59.314184 -1.885816) (end 57.9 -1.3)
       (stroke (width 0.1) (type default)) (layer "Edge.Cuts"))
-    (fp_arc (start 75.062815 -81.787437) (mid 80.012606 -79.737227) (end 82.062814 -74.787436)
+    (fp_arc (start 75.062815 -81.787437) (mid 80.012602 -79.737226) (end 82.062814 -74.787436)
       (stroke (width 0.1) (type solid)) (layer "Edge.Cuts"))
     (fp_arc (start 78.060074 -11.999926) (mid 77.474266 -10.585734) (end 76.060074 -9.999926)
@@
     (fp_arc (start 95.512563 -65.087437) (mid 96.926749 -64.501631) (end 97.512563 -63.087437)
       (stroke (width 0.1) (type default)) (layer "Edge.Cuts"))
-    (fp_arc (start 97.512563 -31.73718) (mid 96.926797 -30.322963) (end 95.512563 -29.73718)
+    (fp_arc (start 97.512563 -31.73718) (mid 96.926803 -30.322928) (end 95.512563 -29.73718)
       (stroke (width 0.1) (type default)) (layer "Edge.Cuts"))
     (fp_line (start 79.925126 -15.45) (end 79.925126 -0.55)
@@
       (net 121 "/IN_O2S") (pinfunction "IN_AUX3") (pintype "passive"))
     (pad "C16" thru_hole circle locked (at 30.815126 -86.685 90) (size 1.7 1.7) (drill 1) (layers "*.Cu" "*.Mask")
-      (net 122 "unconnected-(M1-VR_MAX9924+-PadC16)") (pinfunction "VR_MAX9924+") (pintype "passive+no_connect"))
+      (net 122 "Net-(J2-Pin_1)") (pinfunction "VR_MAX9924+") (pintype "passive"))
     (pad "C16" thru_hole circle locked (at 31.625126 -85.225 90) (size 2 2) (drill 1.2) (layers "*.Cu" "*.Mask")
-      (net 122 "unconnected-(M1-VR_MAX9924+-PadC16)") (pinfunction "VR_MAX9924+") (pintype "passive+no_connect"))
+      (net 122 "Net-(J2-Pin_1)") (pinfunction "VR_MAX9924+") (pintype "passive"))
     (pad "C17" thru_hole circle locked (at 35.825126 -85.225 90) (size 2 2) (drill 1.2) (layers "*.Cu" "*.Mask")
-      (net 123 "unconnected-(M1-VR_MAX9924--PadC17)") (pinfunction "VR_MAX9924-") (pintype "passive+no_connect"))
+      (net 124 "Net-(J2-Pin_3)") (pinfunction "VR_MAX9924-") (pintype "passive"))
     (pad "C17" thru_hole circle locked (at 36.675126 -86.685 90) (size 1.7 1.7) (drill 1) (layers "*.Cu" "*.Mask")
-      (net 123 "unconnected-(M1-VR_MAX9924--PadC17)") (pinfunction "VR_MAX9924-") (pintype "passive+no_connect"))
+      (net 124 "Net-(J2-Pin_3)") (pinfunction "VR_MAX9924-") (pintype "passive"))
     (pad "C18" thru_hole circle locked (at 39.215126 -86.685 90) (size 1.7 1.7) (drill 1) (layers "*.Cu" "*.Mask")
-      (net 124 "unconnected-(M1-VR_DISCRETE+-PadC18)") (pinfunction "VR_DISCRETE+") (pintype "passive+no_connect"))
+      (net 123 "Net-(J2-Pin_2)") (pinfunction "VR_DISCRETE+") (pintype "passive"))
     (pad "C18" thru_hole circle locked (at 40.025126 -85.225 90) (size 2 2) (drill 1.2) (layers "*.Cu" "*.Mask")
-      (net 124 "unconnected-(M1-VR_DISCRETE+-PadC18)") (pinfunction "VR_DISCRETE+") (pintype "passive+no_connect"))
+      (net 123 "Net-(J2-Pin_2)") (pinfunction "VR_DISCRETE+") (pintype "passive"))
     (pad "C19" thru_hole circle locked (at 44.225126 -85.225 90) (size 2 2) (drill 1.2) (layers "*.Cu" "*.Mask")
-      (net 125 "unconnected-(M1-VR_DISCRETE--PadC19)") (pinfunction "VR_DISCRETE-") (pintype "passive+no_connect"))
+      (net 125 "Net-(J2-Pin_4)") (pinfunction "VR_DISCRETE-") (pintype "passive"))
     (pad "C20" thru_hole circle locked (at 48.425126 -85.225 90) (size 2 2) (drill 1.2) (layers "*.Cu" "*.Mask")
       (net 126 "Net-(M1-EGT-)") (pinfunction "EGT-") (pintype "passive"))

Commit message: upd
Parts:
- removed P_C10, P_C20: Pad, hellen-one-common:PAD-TH
- added J3: 43045-0212, Connector_Molex:Molex_Micro-Fit_3.0_43045-0212_2x01_P3.00mm_Vertical, F.Cu at (225.8, 80.4)
- moved M1 4.84 mm to (50.5, 172.3)
Connections:
- G8 pad 10: unconnected-(G8-Pad10) -> /12V_FROM_MAIN_RELAY
- G8 pad 13: unconnected-(G8-Pad13) -> +5VP
- G8 pad 14: unconnected-(G8-Pad14) -> +5VP
- G8 pad 15: unconnected-(G8-Pad15) -> /12V_FROM_MAIN_RELAY
- G8 pad 3: unconnected-(G8-Pad3) -> +5VP
- G8 pad 4: unconnected-(G8-Pad4) -> +5VP
- G8 pad 5: unconnected-(G8-Pad5) -> /12V_FROM_MAIN_RELAY
- G8 pad 8: unconnected-(G8-Pad8) -> +5VP
- G8 pad 9: unconnected-(G8-Pad9) -> +5VP
- M1 pad C10: Net-(M1-EGT+) -> unconnected-(M1-EGT+-PadC10)
- M1 pad C11: GNDA -> Net-(P_C11-Pin_1)
- M1 pad C12: GNDA -> Net-(P_C12-Pin_1)
- M1 pad C13: GNDA -> Net-(P_C13-Pin_1)
- M1 pad C20: Net-(M1-EGT-) -> unconnected-(M1-EGT--PadC20)
- P_C11 pad 1: GNDA -> Net-(P_C11-Pin_1)
- P_C12 pad 1: GNDA -> Net-(P_C12-Pin_1)
- P_C13 pad 1: GNDA -> Net-(P_C13-Pin_1)
Other:
- copper layers 2 -> 4

Commit message: upd
Parts:
- moved P9 233.5 mm to (40.0, 171.0)
- moved P3 224.9 mm to (40.0, 161.0)
- moved P4 220.5 mm to (40.0, 156.0)
- moved P7 219.8 mm to (40.0, 166.0)
- moved J2 216.1 mm to (37.0, 96.0)
- moved P_C11 213.3 mm to (35.0, 87.0)
- moved P_C12 208.6 mm to (39.0, 87.0)
- moved P_C13 203.9 mm to (43.0, 87.0)
- moved P12 200.4 mm to (35.0, 60.1)
- moved P2 193.7 mm to (39.0, 60.1)
- moved F12 189.1 mm to (35.0, 53.1), turned to -90 degrees
- moved P5 183.8 mm to (48.0, 60.1)
- moved P6 180.6 mm to (51.0, 60.1)
- moved P8 179.5 mm to (57.0, 60.1)
- moved P19 178.4 mm to (57.0, 53.1)
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Connections:
- M1 pad C10: unconnected-(M1-EGT+-PadC10) -> /EGT+
- M1 pad C20: unconnected-(M1-EGT--PadC20) -> /EGT-

Commit message: upd
Parts:
- moved Q1 110.9 mm to (103.0, 61.0), turned to 180 degrees
- moved D1 108.7 mm to (114.5, 59.6), turned to -90 degrees
- moved C1 92.6 mm to (114.5, 64.8), turned to 90 degrees
- moved R1 88.7 mm to (110.5, 59.0), turned to -90 degrees
- moved D2 84.5 mm to (119.3, 59.0), turned to 180 degrees
- moved R25 81.3 mm to (117.5, 65.0), turned to -90 degrees
- moved R54 45.5 mm to (124.5, 53.0), turned to 90 degrees
- moved P63 12.2 mm to (160.5, 63.0)
- moved P_C13 12.2 mm to (31.2, 83.8)
- moved P_C11 7.04 mm to (41.2, 83.8)
- moved R51 5.10 mm to (164.0, 61.1)
- moved R64 5.08 mm to (164.0, 53.0)
- moved P60 4.62 mm to (145.2, 55.2)
- moved R49_51 4.61 mm to (155.5, 61.1)
- moved R62_64 4.59 mm to (155.5, 53.0)
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Connections:
- M1 pad C11: Net-(P_C11-Pin_1) -> GNDA
- M1 pad C12: Net-(P_C12-Pin_1) -> GNDA
- M1 pad C13: Net-(P_C13-Pin_1) -> GNDA
- P_C11 pad 1: Net-(P_C11-Pin_1) -> GNDA
- P_C12 pad 1: Net-(P_C12-Pin_1) -> GNDA
- P_C13 pad 1: Net-(P_C13-Pin_1) -> GNDA
Routing:
- net /EGT-: track 0.00 -> 93.1 mm
- net /EGT+: track 0.00 -> 92.2 mm
- net /CANH: track 0.00 -> 69.9 mm
- net /CANL: track 0.00 -> 67.1 mm
- net Net-(J1-Pin_4): track 0.00 -> 66.4 mm
- net Net-(J1-Pin_1): track 0.00 -> 66.4 mm
- net Net-(J2-Pin_4): track 0.00 -> 58.6 mm
- net Net-(J2-Pin_3): track 0.00 -> 54.4 mm
- net Net-(J2-Pin_2): track 0.00 -> 53.2 mm
- net Net-(J2-Pin_1): track 0.00 -> 47.8 mm
- net /OUT_TACH: track 0.00 -> 35.8 mm
- net Net-(M1-DC2_PWM): track 0.00 -> 34.5 mm
- net Net-(J1-Pin_5): track 0.00 -> 33.3 mm
- net Net-(J1-Pin_2): track 0.00 -> 28.3 mm
- net /3X: track 0.00 -> 27.4 mm
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