File: uaefi-adapter-NA-90-95.kicad_pcb (KiCad board)
At the start: 4 copper layers, 154 x 159 mm, 73 parts, among them J1 43045-0612, J11 Conn_01x01, J13 Conn_01x01, J14 Conn_01x01, J15 Conn_01x01, J16 Conn_01x01, J17 Conn_01x01, J2 43045-0412, J3 43045-0212, M1 Module:uaefi/0.2, P1 178780-1, P10 Pad, P11 Pad, P12 Pad, P19 Pad, P2 Pad, P21 Pad, P3 Pad, P4 Pad, P5 Pad, P55 Pad, P56 Pad, P6 Pad, P60 Pad, P63 Pad, P7 Pad, P8 Pad, P9 Pad, Q1 ZXMS6005SGTA

Commit message: in progress
Routing:
- net /OUT_ETB+: track 0.00 -> 181.0 mm
- net /OUT_ETB-: track 0.00 -> 179.6 mm
- net /OUT_CHECK_ENGINE: track 0.00 -> 82.2 mm
- net /OUT_IGN1: track 0.00 -> 76.7 mm
- net /IN_AC_SW: track 0.00 -> 39.2 mm
- net /IN_VSS: track 0.00 -> 33.1 mm
- net /+12V_PERM: track 0.00 -> 21.8 mm
Changed lines of the file:
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@@
     (fp_arc (start 23 -13) (mid 24.414214 -12.414214) (end 25 -11)
       (stroke (width 0.1) (type default)) (layer "Edge.Cuts"))
-    (fp_arc (start 27 -1.287437) (mid 25.585764 -1.87322) (end 25 -3.287437)
+    (fp_arc (start 27 -1.287437) (mid 25.585777 -1.873212) (end 25 -3.287437)
       (stroke (width 0.1) (type default)) (layer "Edge.Cuts"))
     (fp_arc (start 59.899911 -8.00008) (mid 60.48572 -9.414273) (end 61.899911 -10.00008)
@@
     (fp_arc (start 59.9 -3.3) (mid 59.314184 -1.885816) (end 57.9 -1.3)
       (stroke (width 0.1) (type default)) (layer "Edge.Cuts"))
-    (fp_arc (start 75.062815 -81.787437) (mid 80.0126 -79.737223) (end 82.062814 -74.787436)
+    (fp_arc (start 75.062815 -81.787437) (mid 80.012603 -79.737224) (end 82.062814 -74.787436)
       (stroke (width 0.1) (type solid)) (layer "Edge.Cuts"))
     (fp_arc (start 78.060074 -11.999926) (mid 77.474266 -10.585734) (end 76.060074 -9.999926)
@@
     (fp_arc (start 95.512563 -65.087437) (mid 96.926749 -64.501631) (end 97.512563 -63.087437)
       (stroke (width 0.1) (type default)) (layer "Edge.Cuts"))
-    (fp_arc (start 97.512563 -31.73718) (mid 96.926797 -30.322963) (end 95.512563 -29.73718)
+    (fp_arc (start 97.512563 -31.73718) (mid 96.926803 -30.322928) (end 95.512563 -29.73718)
       (stroke (width 0.1) (type default)) (layer "Edge.Cuts"))
     (fp_line (start 79.925126 -15.45) (end 79.925126 -0.55)
@@
   (segment (start 47.75 39.25938) (end 47.75 51.19) (width 0.25) (layer "F.Cu") (net 28))
   (segment (start 49.089381 37.919999) (end 47.75 39.25938) (width 0.25) (layer "F.Cu") (net 28))
+  (segment (start 29.5 99.75) (end 33.912437 104.162437) (width 0.25) (layer "F.Cu") (net 29))
+  (segment (start 33.912437 104.162437) (end 59.665126 104.162437) (width 0.25) (layer "F.Cu") (net 29))
+  (segment (start 44.75 63) (end 29.5 78.25) (width 0.25) (layer "F.Cu") (net 29))
+  (segment (start 59.665126 104.162437) (end 60.840126 105.337437) (width 0.25) (layer "F.Cu") (net 29))
+  (segment (start 29.5 78.25) (end 29.5 99.75) (width 0.25) (layer "F.Cu") (net 29))
   (segment (start 46.089641 57.850359) (end 44.75 59.19) (width 0.25) (layer "F.Cu") (net 30))
   (segment (start 46.089641 42.420879) (end 46.089641 57.850359) (width 0.25) (layer "F.Cu") (net 30))
@@
   (segment (start 153.75 126.75) (end 153.75 105.5) (width 0.25) (layer "F.Cu") (net 45))
   (segment (start 155.25 128.25) (end 153.75 126.75) (width 0.25) (layer "F.Cu") (net 45))
+  (segment (start 43.449999 28.05) (end 29.3 42.199999) (width 0.25) (layer "B.Cu") (net 91))
+  (segment (start 70.561396 28.05) (end 43.449999 28.05) (width 0.25) (layer "B.Cu") (net 91))
+  (segment (start 76.140721 33.629325) (end 70.561396 28.05) (width 0.25) (layer "B.Cu") (net 91))
+  (segment (start 38.75 128.537311) (end 56.800126 146.587437) (width 0.25) (layer "B.Cu") (net 91))
+  (segment (start 38.75 110.5) (end 38.75 128.537311) (width 0.25) (layer "B.Cu") (net 91))
+  (segment (start 76.140721 42.420879) (end 76.140721 33.629325) (width 0.25) (layer "B.Cu") (net 91))
+  (segment (start 29.3 101.05) (end 38.75 110.5) (width 0.25) (layer "B.Cu") (net 91))
+  (segment (start 29.3 42.199999) (end 29.3 101.05) (width 0.25) (layer "B.Cu") (net 91))
+  (segment (start 73.140981 31.265981) (end 70.375 28.5) (width 0.25) (layer "B.Cu") (net 93))
+  (segment (start 70.375 28.5) (end 43.75 28.5) (width 0.25) (layer "B.Cu") (net 93))
+  (segment (start 39.2 126.868037) (end 58.9194 146.587437) (width 0.25) (layer "B.Cu") (net 93))
+  (segment (start 58.9194 146.587437) (end 62.300126 146.587437) (width 0.25) (layer "B.Cu") (net 93))
+  (segment (start 39.2 110.313604) (end 39.2 126.868037) (width 0.25) (layer "B.Cu") (net 93))
+  (segment (start 29.75 100.863604) (end 39.2 110.313604) (width 0.25) (layer "B.Cu") (net 93))
+  (segment (start 73.140981 42.420879) (end 73.140981 31.265981) (width 0.25) (layer "B.Cu") (net 93))
+  (segment (start 43.75 28.5) (end 29.75 42.5) (width 0.25) (layer "B.Cu") (net 93))
+  (segment (start 29.75 42.5) (end 29.75 100.863604) (width 0.25) (layer "B.Cu") (net 93))
+  (segment (start 29.05 101.55) (end 54.687437 127.187437) (width 0.25) (layer "F.Cu") (net 95))
+  (segment (start 29.05 75.7) (end 29.05 101.55) (width 0.25) (layer "F.Cu") (net 95))
+  (segment (start 41.75 63) (end 29.05 75.7) (width 0.25) (layer "F.Cu") (net 95))
+  (segment (start 54.687437 127.187437) (end 56.800126 127.187437) (width 0.25) (layer "F.Cu") (net 95))
+  (segment (start 70.212689 72.75) (end 79.125126 81.662437) (width 0.25) (layer "F.Cu") (net 108))
+  (segment (start 53.75 63) (end 63.5 72.75) (width 0.25) (layer "F.Cu") (net 108))
+  (segment (start 63.5 72.75) (end 70.212689 72.75) (width 0.25) (layer "F.Cu") (net 108))
+  (segment (start 81.062689 71) (end 91.725126 81.662437) (width 0.25) (layer "F.Cu") (net 110))
+  (segment (start 60.25 63) (end 68.25 71) (width 0.25) (layer "F.Cu") (net 110))
+  (segment (start 68.25 71) (end 81.062689 71) (width 0.25) (layer "F.Cu") (net 110))
   (segment (start 77.536343 88.75122) (end 79.125126 87.162437) (width 0.25) (layer "F.Cu") (net 114))
   (segment (start 42.24878 88.75122) (end 77.536343 88.75122) (width 0.25) (layer "F.Cu") (net 114))
@@
   (segment (start 67.189421 42.420879) (end 67.189421 45.689421) (width 0.25) (layer "F.Cu") (net 142))
   (segment (start 67.189421 45.689421) (end 70.25 48.75) (width 0.25) (layer "F.Cu") (net 142))
+  (segment (start 36.490981 44.990981) (end 36.490981 42.420879) (width 0.5) (layer "F.Cu") (net 143))
+  (segment (start 34 60.25) (end 36.75 57.5) (width 0.5) (layer "F.Cu") (net 143))
+  (segment (start 36.75 45.25) (end 36.490981 44.990981) (width 0.5) (layer "F.Cu") (net 143))
+  (segment (start 36.75 57.5) (end 36.75 45.25) (width 0.5) (layer "F.Cu") (net 143))
+  (segment (start 34 63) (end 34 60.25) (width 0.5) (layer "F.Cu") (net 143))
   (segment (start 130.391581 37.919999) (end 129 39.31158) (width 0.25) (layer "F.Cu") (net 144))
   (segment (start 129 39.31158) (end 129 55.25) (width 0.25) (layer "F.Cu") (net 144))

Commit message: upd
Parts:
- moved R49_51 0.91 mm to (155.5, 62.0)
- moved R51 0.91 mm to (164.0, 62.0)
- moved P63 0.50 mm to (160.5, 63.5)
Routing:
- net /OUT_INJ2: track 14.8 -> 341.7 mm
- net /OUT_INJ1: track 18.4 -> 330.1 mm
- net /OUT_INJ3: track 0.00 -> 267.4 mm
- net /OUT_INJ4: track 0.00 -> 266.6 mm
- net /OUT_PUMP_RELAY: track 0.00 -> 148.8 mm, vias 0 -> 2
- net /OUT_IDLE: track 0.00 -> 133.8 mm, vias 0 -> 1
- net /OUT_VVT: track 0.00 -> 130.4 mm, vias 0 -> 1
- net /CANL: track 67.1 -> 194.3 mm, vias 0 -> 1
- net /CANH: track 69.9 -> 195.3 mm, vias 0 -> 1
- net /OUT_CONDENSER_FAN: track 0.00 -> 116.2 mm, vias 0 -> 1
- net /IN_TPS1: track 0.00 -> 107.5 mm, vias 0 -> 1
- net /WBO_Vs/Ip: track 0.00 -> 105.5 mm
- net /OUT_BOOST_CONTROL: track 0.00 -> 98.8 mm
- net /IN_CAM: track 0.00 -> 94.8 mm, vias 0 -> 1
- net /WBO_H-: track 0.00 -> 92.6 mm
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- added copper zone on F.Cu, net Net-(D1-A)
