File: uaefi-adapter-NA-90-95.kicad_pcb (KiCad board)
At the start: 4 copper layers, 154 x 159 mm, 73 parts, among them J1 43045-0612, J11 Conn_01x01, J13 Conn_01x01, J14 Conn_01x01, J15 Conn_01x01, J16 Conn_01x01, J17 Conn_01x01, J2 43045-0412, J3 43045-0212, M1 Module:uaefi/0.2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

Commit message: upd
Parts:
- moved F32 10.8 mm to (106.0, 53.1)
Routing:
- net /12V_FROM_MAIN_RELAY: track 0.00 -> 243.8 mm, vias 0 -> 4
- net +5VP: track 0.00 -> 186.0 mm, vias 0 -> 2
- net /TACH: track 0.00 -> 184.6 mm, vias 0 -> 4
- net GNDA: track 0.00 -> 158.7 mm
- net /2D: track 13.5 -> 18.2 mm
- net /OUT_INJ4: track 266.6 -> 267.9 mm
- net /OUT_INJ3: track 267.4 -> 268.3 mm
- net /IN_CLT: track 51.9 -> 52.5 mm
- net GND: vias 0 -> 60
- added copper zone on F.Cu, net +5VP
- added copper zone on B.Cu, net GND
- added copper zone on F.Cu, net GND
- added copper zone on In1.Cu, net GND
- added copper zone on In2.Cu, net GND

Commit message: upd
Other:
- board text added: "+12V"
- board text added: "GNDA"
