File: uaefi-adapter-NA-90-95.kicad_pcb (KiCad board)
At the start: 4 copper layers, 154 x 159 mm, 73 parts, among them J1 43045-0612, J11 Conn_01x01, J13 Conn_01x01, J14 Conn_01x01, J15 Conn_01x01, J16 Conn_01x01, J17 Conn_01x01, J2 43045-0412, J3 43045-0212, M1 Module:uaefi/0.2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

Commit message: rev b
Routing:
- net GND: vias 60 -> 66
Other:
- outline, holes or cut-outs redrawn
- board text added: "COMMUNITY SUPPORT ECU https://rusefi.com/s/community https://rusefi.com/s/uaefi-NA rev. b"
- board text removed: "COMMUNITY SUPPORT ECU https://rusefi.com/s/community https://rusefi.com/s/uaefi-NA"

Commit message: #18 #19
Routing:
- net /WBO_H-: track 92.6 -> 153.7 mm
- net +5VP: track 186.0 -> 187.6 mm
- net /OUT_BOOST_CONTROL: track 98.8 -> 98.0 mm
- net /OUT_IDLE: track 133.8 -> 134.4 mm
- net /OUT_RADIATOR_FAN_RELAY: track 62.1 -> 61.6 mm
Other:
- board text added: "COMMUNITY SUPPORT ECU https://rusefi.com/s/community https://rusefi.com/s/uaefi-NA uaefi NA6 adapter rev. b"
- board text removed: "COMMUNITY SUPPORT ECU https://rusefi.com/s/community https://rusefi.com/s/uaefi-NA rev. b"
